File: etutti/hardware/kicad/etuttino.kicad_pcb (KiCad board)
At the start: 2 copper layers, 183.4 x 132.2 mm, 123 parts, among them J1 PinSocket_1x14_P2.54mm_Vertic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, J2 PinSocket_1x14_P2.54mm_Vertic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, SW1 Gateron_Magnetic_MX_1u, SW10 Gateron_Magnetic_MX_1u, SW11 Gateron_Magnetic_MX_1u, SW12 Gateron_Magnetic_MX_1u, SW13 Gateron_Magnetic_MX_1u, SW14 Gateron_Magnetic_MX_1u, SW15 Gateron_Magnetic_MX_1u, SW16 Gateron_Magnetic_MX_1u, SW17 Gateron_Magnetic_MX_1u, SW18 Gateron_Magnetic_MX_1u, SW19 Gateron_Magnetic_MX_1u, SW2 Gateron_Magnetic_MX_1u, SW20 Gateron_Magnetic_MX_1u, SW21 Gateron_Magnetic_MX_1u, SW22 Gateron_Magnetic_MX_1u, SW23 Gateron_Magnetic_MX_1u, SW24 Gateron_Magnetic_MX_1u, SW25 Gateron_Magnetic_MX_1u, SW26 Gateron_Magnetic_MX_1u, SW27 Gateron_Magnetic_MX_1u, SW28 Gateron_Magnetic_MX_1u, SW29 Gateron_Magnetic_MX_1u, SW3 Gateron_Magnetic_MX_1u, SW30 Gateron_Magnetic_MX_1u, SW31 Gateron_Magnetic_MX_1u, SW32 Gateron_Magnetic_MX_1u, SW33 Gateron_Magnetic_MX_1u, SW34 Gateron_Magnetic_MX_1u, SW4 Gateron_Magnetic_MX_1u, SW5 Gateron_Magnetic_MX_1u, SW6 Gateron_Magnetic_MX_1u, SW7 Gateron_Magnetic_MX_1u, SW8 Gateron_Magnetic_MX_1u, SW9 Gateron_Magnetic_MX_1u, U1 DRV5056A3QDBZR, U10 DRV5056A3QDBZR, U11 DRV5056A3QDBZR, U12 DRV5056A3QDBZR, U13 DRV5056A3QDBZR, U14 DRV5056A3QDBZR, U15 DRV5056A3QDBZR, U16 DRV5056A3QDBZR, U17 DRV5056A3QDBZR, U18 DRV5056A3QDBZR, U19 DRV5056A3QDBZR, U2 DRV5056A3QDBZR, U20 DRV5056A3QDBZR, U21 DRV5056A3QDBZR, U22 DRV5056A3QDBZR, U23 DRV5056A3QDBZR, U24 DRV5056A3QDBZR, U25 DRV5056A3QDBZR, U26 DRV5056A3QDBZR, U27 DRV5056A3QDBZR, U28 DRV5056A3QDBZR, U29 DRV5056A3QDBZR, U3 DRV5056A3QDBZR, U30 DRV5056A3QDBZR, U31 DRV5056A3QDBZR, U32 DRV5056A3QDBZR, U33 DRV5056A3QDBZR, U34 DRV5056A3QDBZR, U4 DRV5056A3QDBZR, U41 CD74HC4067M96, U42 CD74HC4067M96, U43 CD74HC4067M96, U5 DRV5056A3QDBZR, U50 AMS1117-3.3, U6 DRV5056A3QDBZR, U7 DRV5056A3QDBZR, U8 DRV5056A3QDBZR, U9 DRV5056A3QDBZR

Commit message: eTuttino: Castagnari Magica K2 layout, slim board, browser sound, manual visuals
- Layout: 41 keys like the Castagnari Magica K2 treble keyboard (rows
  A3..D#6, G3..G6, G#3..D6, A3..C5), on the page, in the firmware and on
  the board; computer-keyboard mapping extended (ABNT2), legends from
  navigator.keyboard.getLayoutMap() where available.
- Board 267 x 88.2 mm, only the four key rows tall: the Teensy + Audio
  Board stack sits in the corner row 4 leaves free (USB and headphone
  jack at the right edge), Audio Board soldered low so the stack (~17 mm)
  stays below the keycaps (~19 mm); plate notched; muxes behind row 4.
  Router: power buses joined by the router, critical nets before the
  sensor outputs, retry with the failed net first, layer changes next to
  an existing via reuse it. DRC 0/0/0, firmware cross-check 41/41.
- "Listen in this browser" (websynth.js): the eTuttino's sounds through
  the computer's speakers, off until the user switches it on; same CCs
  as the firmware.
- Manuals rewritten for the new board in en/pt/es, with 3D renders
  (assembly3d.py: simple VRML switches, keycaps, plate, Teensy, Audio
  Board) and close-ups; click opens the full-resolution image.

Co-Authored-By: Claude Opus 5.5 <noreply@anthropic.com>
Parts:
- removed C42, C43: 100nF, C_0805_2012Metric
- removed C50: 10uF, C_0805_2012Metric
- removed C51: 22uF, C_0805_2012Metric
- removed U42, U43: CD74HC4067M96, SOIC-24W_7.5x15.4mm_P1.27mm
- removed U50: AMS1117-3.3, SOT-223-3_TabPin2
- added C35: 100nF, C_0805_2012Metric, B.Cu at (215.6, 31.6)
- added C36: 100nF, C_0805_2012Metric, B.Cu at (25.1, 12.5)
- added C37: 100nF, C_0805_2012Metric, B.Cu at (44.1, 12.5)
- added C38: 100nF, C_0805_2012Metric, B.Cu at (63.1, 12.5)
- added C39: 100nF, C_0805_2012Metric, B.Cu at (82.2, 12.5)
- added C40: 100nF, C_0805_2012Metric, B.Cu at (101.2, 12.5)
- added C71: 100nF, C_0805_2012Metric, B.Cu at (149.7, 26.3)
- added C72: 100nF, C_0805_2012Metric, B.Cu at (179.7, 26.3)
- added C73: 100nF, C_0805_2012Metric, B.Cu at (209.2, 26.3)
- added C80: 10uF, C_0805_2012Metric, B.Cu at (254.0, 26.7)
- added C81: 22uF, C_0805_2012Metric, B.Cu at (239.8, 26.7)
- added H11: MountingHole_2.2mm_M2, MountingHole_2.2mm_M2, F.Cu at (264.0, 85.2)
- added H12: MountingHole_2.2mm_M2, MountingHole_2.2mm_M2, F.Cu at (264.0, 43.8)
- added SW35: Gateron_Magnetic_MX_1u, Gateron_Magnetic_MX_1u, F.Cu at (215.6, 34.6)
- added SW36: Gateron_Magnetic_MX_1u, Gateron_Magnetic_MX_1u, F.Cu at (25.1, 15.5)
- added SW37: Gateron_Magnetic_MX_1u, Gateron_Magnetic_MX_1u, F.Cu at (44.1, 15.5)
- added SW38: Gateron_Magnetic_MX_1u, Gateron_Magnetic_MX_1u, F.Cu at (63.1, 15.5)
- added SW39: Gateron_Magnetic_MX_1u, Gateron_Magnetic_MX_1u, F.Cu at (82.2, 15.5)
- added SW40: Gateron_Magnetic_MX_1u, Gateron_Magnetic_MX_1u, F.Cu at (101.2, 15.5)
- added SW41: Gateron_Magnetic_MX_1u, Gateron_Magnetic_MX_1u, F.Cu at (120.3, 15.5)
- added U35: DRV5056A3QDBZR, SOT-23-3, B.Cu at (215.6, 34.6)
- added U36: DRV5056A3QDBZR, SOT-23-3, B.Cu at (25.1, 15.5)
- added U37: DRV5056A3QDBZR, SOT-23-3, B.Cu at (44.1, 15.5)
- added U38: DRV5056A3QDBZR, SOT-23-3, B.Cu at (63.1, 15.5)
- added U39: DRV5056A3QDBZR, SOT-23-3, B.Cu at (82.2, 15.5)
- added U40: DRV5056A3QDBZR, SOT-23-3, B.Cu at (101.2, 15.5)
- added U51: CD74HC4067M96, SOIC-24W_7.5x15.4mm_P1.27mm, B.Cu at (147.3, 16.5)
- added U52: CD74HC4067M96, SOIC-24W_7.5x15.4mm_P1.27mm, B.Cu at (177.3, 16.5)
- added U53: CD74HC4067M96, SOIC-24W_7.5x15.4mm_P1.27mm, B.Cu at (206.8, 16.5)
- added U60: AMS1117-3.3, SOT-223-3_TabPin2, B.Cu at (247.0, 23.5)
- U41: value CD74HC4067M96 -> DRV5056A3QDBZR; footprint SOIC-24W_7.5x15.4mm_P1.27mm -> SOT-23-3
- moved H5 257.4 mm to (256.6, 85.2)
- moved H3 224.0 mm to (222.7, 3.00)
- moved H2 195.6 mm to (3.00, 85.2)
- moved H6 178.9 mm to (10.8, 72.7)
- moved C10 163.8 mm to (196.5, 69.7)
- moved C11 163.8 mm to (215.6, 69.7)
- moved SW10 163.8 mm to (196.5, 72.7)
- moved SW11 163.8 mm to (215.6, 72.7)
- moved U10 163.8 mm to (196.5, 72.7)
- moved U11 163.8 mm to (215.6, 72.7)
- moved C9 163.8 mm to (177.4, 69.7)
- moved SW9 163.8 mm to (177.4, 72.7)
- moved U9 163.8 mm to (177.4, 72.7)
- moved C25 140.4 mm to (25.1, 31.6)
- moved SW25 140.4 mm to (25.1, 34.6)
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Connections:
- U41 pad 1: COM0 -> VCC
- U41 pad 2: (no net) -> OUT_U41
- U41 pad 3: (no net) -> GND
Routing:
- net OUT_U35: track 0.00 -> 236.9 mm, vias 0 -> 7
- net OUT_U40: track 0.00 -> 187.8 mm, vias 0 -> 10
- net OUT_U33: track 48.5 -> 208.5 mm, vias 4 -> 9
- net OUT_U32: track 48.0 -> 183.2 mm, vias 2 -> 6
- net OUT_U22: track 65.7 -> 190.4 mm, vias 2 -> 6
- net OUT_U36: track 0.00 -> 122.3 mm, vias 0 -> 4
- net GND: track 1230.9 -> 1351.5 mm, vias 14 -> 13
- net OUT_U37: track 0.00 -> 119.8 mm, vias 0 -> 6
- net OUT_U31: track 53.1 -> 153.3 mm, vias 2 -> 10
- net OUT_U39: track 0.00 -> 96.9 mm, vias 0 -> 6
- net OUT_U38: track 0.00 -> 91.1 mm, vias 0 -> 2
- net OUT_U41: track 0.00 -> 84.4 mm, vias 0 -> 4
- net OUT_U12: track 81.6 -> 144.5 mm
- net OUT_U25: track 73.3 -> 130.3 mm, vias 4 -> 2
- net OUT_U27: track 41.5 -> 97.2 mm
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Other:
- board size 183.4 x 132.2 mm -> 267 x 88.2 mm
- board text added: "Sensors DRV5056A3 on this side, under each switch"
- board text added: "Teensy 4.0 on Audio Board Rev D - USB + jack >"
- board text added: "eTuttino v0.3 HE"
- board text added: "eTuttino v0.3 HE - Magica K2 layout, C-griff G3-G6 - beatconfused.com/etutti"
- board text removed: "Sensors DRV5056A3, back side, under each switch"
- board text removed: "Teensy 4.0 + Audio Board Rev D"
- board text removed: "USB >"
- board text removed: "beatconfused.com/etutti"
- board text removed: "eTuttino v0.2 HE"
- board text removed: "eTuttino v0.2 HE - C-griff G3-G5"

Commit message: eTuttino: 44-key layout, power LED, muxes spread out, no brand reference
- Row 2 now ends at E6 (12 keys); row 4 runs A3..C6 (10 keys) on row 2's
  columns (A3 above A#3, C6 above C#6); row 1 unchanged.
- Bicolour power LED D1 (pins 4/5 via R1/R2 330R): orange while the keys
  are first read, green playing, red blinking on codec/sensor errors.
- Multiplexers: U51 front-right corner, U53 back-left corner, U52 beside
  the Teensy. The router picks each sensor's mux channel and writes
  KEY_INPUT into the sketch; the far mux's long lines route last.
- High-note reed tables in the firmware (the full tables aliased).
- Board DRC 0/0/0, firmware cross-check 44/44; renders and manuals
  (en/pt/es) updated, incl. a U53 close-up.
- Removed every mention of the commercial accordion layout reference.

Co-Authored-By: Claude Opus 5.5 <noreply@anthropic.com>
Parts:
- removed H12: MountingHole_2.2mm_M2, MountingHole_2.2mm_M2
- added C42: 100nF, C_0805_2012Metric, B.Cu at (167.9, 12.5)
- added C43: 100nF, C_0805_2012Metric, B.Cu at (187.0, 12.5)
- added C44: 100nF, C_0805_2012Metric, B.Cu at (206.0, 12.5)
- added D1: LED 3mm red/green CC, LED_D3.0mm-3, F.Cu at (254.5, 82.0)
- added R1: 330, R_0805_2012Metric, B.Cu at (255.2, 77.5)
- added R2: 330, R_0805_2012Metric, B.Cu at (262.0, 77.5)
- added SW42: Gateron_Magnetic_MX_1u, Gateron_Magnetic_MX_1u, F.Cu at (167.9, 15.5)
- added SW43: Gateron_Magnetic_MX_1u, Gateron_Magnetic_MX_1u, F.Cu at (187.0, 15.5)
- added SW44: Gateron_Magnetic_MX_1u, Gateron_Magnetic_MX_1u, F.Cu at (206.0, 15.5)
- added U42: DRV5056A3QDBZR, SOT-23-3, B.Cu at (167.9, 15.5)
- added U43: DRV5056A3QDBZR, SOT-23-3, B.Cu at (187.0, 15.5)
- added U44: DRV5056A3QDBZR, SOT-23-3, B.Cu at (206.0, 15.5)
- moved C24 219.9 mm to (25.1, 31.6)
- moved SW24 219.9 mm to (25.1, 34.6)
- moved U24 219.9 mm to (25.1, 34.6)
- moved U53 191.8 mm to (15.0, 15.5), turned to 180 degrees
- moved C73 190.8 mm to (19.6, 5.12)
- moved C35 182.0 mm to (34.6, 12.5)
- moved SW35 182.0 mm to (34.6, 15.5)
- moved U35 182.0 mm to (34.6, 15.5)
- moved C71 114.0 mm to (252.4, 75.8)
- moved U51 114.0 mm to (250.0, 66.0)
- moved H9 86.0 mm to (220.6, 15.5)
- moved H10 83.4 mm to (264.0, 85.2)
- moved U52 69.5 mm to (246.5, 9.50), turned to -90 degrees
- moved C72 59.2 mm to (236.5, 9.50), turned to -90 degrees
- moved H11 37.4 mm to (264.0, 47.8)
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Connections:
- C72 pad 1: VCC -> GND
- C72 pad 2: GND -> VCC
- C73 pad 1: VCC -> GND
- C73 pad 2: GND -> VCC
- J1 pad 6: (no net) -> LED_R_DRV
- J1 pad 7: (no net) -> LED_G_DRV
- U51 pad 16: OUT_U15 -> OUT_U19
- U51 pad 17: OUT_U3 -> OUT_U8
- U51 pad 18: OUT_U27 -> OUT_U20
- U51 pad 19: OUT_U38 -> OUT_U21
- U51 pad 2: OUT_U2 -> OUT_U23
- U51 pad 20: OUT_U14 -> OUT_U22
- U51 pad 21: (no net) -> OUT_U11
- U51 pad 22: (no net) -> OUT_U10
- U51 pad 23: (no net) -> OUT_U9
- U51 pad 3: OUT_U26 -> OUT_U7
- U51 pad 4: OUT_U37 -> OUT_U4
- U51 pad 5: OUT_U13 -> OUT_U1
- U51 pad 6: OUT_U1 -> OUT_U2
- U51 pad 7: OUT_U25 -> OUT_U3
- U51 pad 8: OUT_U36 -> OUT_U5
- U51 pad 9: OUT_U12 -> OUT_U6
- U52 pad 16: OUT_U7 -> (no net)
- U52 pad 17: OUT_U31 -> (no net)
- U52 pad 18: OUT_U18 -> OUT_U34
- U52 pad 19: OUT_U6 -> OUT_U33
- U52 pad 2: OUT_U17 -> OUT_U40
- U52 pad 20: OUT_U30 -> OUT_U31
- U52 pad 21: OUT_U41 -> OUT_U30
- U52 pad 22: (no net) -> OUT_U29
- U52 pad 23: (no net) -> OUT_U18
- U52 pad 3: OUT_U5 -> OUT_U41
- U52 pad 4: OUT_U29 -> OUT_U32
- U52 pad 5: OUT_U40 -> OUT_U42
- U52 pad 6: OUT_U16 -> OUT_U43
- U52 pad 7: OUT_U4 -> OUT_U44
- U52 pad 8: OUT_U28 -> (no net)
- U52 pad 9: OUT_U39 -> (no net)
- U53 pad 16: OUT_U24 -> OUT_U14
- U53 pad 17: OUT_U23 -> OUT_U13
- U53 pad 18: OUT_U11 -> OUT_U37
- U53 pad 19: OUT_U35 -> OUT_U25
- U53 pad 2: OUT_U34 -> OUT_U26
- U53 pad 20: OUT_U22 -> OUT_U12
- U53 pad 21: OUT_U10 -> OUT_U36
- U53 pad 22: (no net) -> OUT_U24
- U53 pad 23: (no net) -> OUT_U35
- U53 pad 3: OUT_U21 -> OUT_U38
- U53 pad 4: OUT_U9 -> OUT_U27
- U53 pad 5: OUT_U33 -> OUT_U39
- U53 pad 6: OUT_U20 -> OUT_U15
- U53 pad 7: OUT_U8 -> OUT_U28
- U53 pad 8: OUT_U32 -> OUT_U16
- U53 pad 9: OUT_U19 -> OUT_U17
Routing:
- net SEL2: track 99.7 -> 312.3 mm, vias 4 -> 3
- net SEL3: track 108.2 -> 311.1 mm, vias 4 -> 10
- net SEL1: track 117.7 -> 319.9 mm, vias 0 -> 7
- net OUT_U6: track 87.0 -> 280.8 mm, vias 2 -> 8
- net COM2: track 35.9 -> 226.1 mm, vias 1 -> 5
- net SEL0: track 118.7 -> 308.6 mm, vias 1 -> 4
- net OUT_U35: track 236.9 -> 60.1 mm, vias 7 -> 8
- net OUT_U5: track 97.8 -> 256.7 mm, vias 2 -> 7
- net OUT_U33: track 208.5 -> 61.9 mm, vias 9 -> 6
- net VCC: track 990.8 -> 1119.3 mm
- net OUT_U22: track 190.4 -> 63.6 mm, vias 6 -> 4
- net OUT_U32: track 183.2 -> 81.7 mm, vias 6 -> 4
- net OUT_U12: track 144.5 -> 48.0 mm
- net OUT_U42: track 0.00 -> 89.6 mm, vias 0 -> 4
- net OUT_U2: track 120.4 -> 205.1 mm, vias 2 -> 4
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Other:
- board text added: "POWER"
- board text added: "eTuttino v0.4 HE"
- board text added: "eTuttino v0.4 HE - C-griff G3-E6 - beatconfused.com/etutti"
- board text removed: "eTuttino v0.3 HE"
- board text removed: "eTuttino v0.3 HE - Magica K2 layout, C-griff G3-G6 - beatconfused.com/etutti"

Commit message: eTuttino: Teensy stack on the left, 3D-printed case, stiffer board
- Ergonomic layout: the Teensy + Audio Board sit in the back-left corner,
  USB and headphone jack facing the left edge (cables away from the
  playing hand). Muxes, LDO and holes follow; the power LED sits just in
  front of the stack, U52 in a new 15 mm back strip. 267 x 97.2 mm,
  rerouted: DRC 0/0/0, firmware check 44/44 (KEY_INPUT updated, flashed).
- Case: case.py (FreeCAD) builds a tray + top shell (STL/STEP in fab/):
  stepped key opening, LED window, pod over the stack with USB/jack
  openings. case_check.py proves it touches no keycap over its travel,
  no switch and nothing of the stack.
- Stiffness: mechanics.py puts 43 pillars in the tray where the back of
  the board has only traces, and estimates the sag under a 3 N press
  (2.6 mm on the mounting holes alone, 0.027 mm in the case).
- Renders: all 28 stacking-header legs through the board with solder,
  the Teensy's pin spacers and tips, switch bases on the board, the
  finished case, the tray. Manuals (en/pt/es) and README updated, with
  where to get the case printed.

Co-Authored-By: Claude Opus 5.5 <noreply@anthropic.com>
Parts:
- moved H1 261.2 mm to (264.0, 12.0)
- moved H10 261.2 mm to (3.00, 94.2)
- moved H11 261.2 mm to (3.00, 56.8)
- moved H2 261.2 mm to (264.0, 94.2)
- moved J1 256.8 mm to (5.50, 39.6), turned to 90 degrees
- moved J2 256.2 mm to (5.50, 24.4), turned to 90 degrees
- moved H6 245.6 mm to (256.2, 81.7)
- moved H7 245.6 mm to (256.2, 43.6)
- moved C80 241.0 mm to (13.0, 28.8)
- moved D1 238.7 mm to (17.0, 58.0)
- moved R1 238.7 mm to (17.7, 53.5)
- moved R2 238.7 mm to (24.5, 53.5)
- moved U53 237.2 mm to (252.0, 24.5)
- moved C73 236.6 mm to (254.4, 34.3)
- moved C71 233.2 mm to (19.4, 84.8)
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Connections:
- C80 pad 1: VIN -> GND
- C80 pad 2: GND -> VIN
- C81 pad 1: VCC -> GND
- C81 pad 2: GND -> VCC
- U51 pad 16: OUT_U19 -> OUT_U12
- U51 pad 17: OUT_U8 -> OUT_U13
- U51 pad 18: OUT_U20 -> OUT_U14
- U51 pad 19: OUT_U21 -> OUT_U15
- U51 pad 2: OUT_U23 -> OUT_U5
- U51 pad 20: OUT_U22 -> OUT_U4
- U51 pad 21: OUT_U11 -> OUT_U3
- U51 pad 22: OUT_U10 -> OUT_U2
- U51 pad 23: OUT_U9 -> OUT_U1
- U51 pad 3: OUT_U7 -> OUT_U6
- U51 pad 4: OUT_U4 -> OUT_U7
- U51 pad 5: OUT_U1 -> OUT_U8
- U51 pad 6: OUT_U2 -> OUT_U9
- U51 pad 7: OUT_U3 -> OUT_U11
- U51 pad 8: OUT_U5 -> OUT_U10
- U51 pad 9: OUT_U6 -> OUT_U16
- U52 pad 18: OUT_U34 -> (no net)
- U52 pad 19: OUT_U33 -> OUT_U17
- U52 pad 2: OUT_U40 -> OUT_U39
- U52 pad 20: OUT_U31 -> (no net)
- U52 pad 21: OUT_U30 -> OUT_U27
- U52 pad 22: OUT_U29 -> OUT_U28
- U52 pad 23: OUT_U18 -> OUT_U29
- U52 pad 3: OUT_U41 -> OUT_U38
- U52 pad 4: OUT_U32 -> OUT_U26
- U52 pad 5: OUT_U42 -> OUT_U24
- U52 pad 6: OUT_U43 -> OUT_U37
- U52 pad 7: OUT_U44 -> OUT_U25
- U52 pad 8: (no net) -> OUT_U36
- U52 pad 9: (no net) -> OUT_U35
- U53 pad 16: OUT_U14 -> OUT_U34
- U53 pad 17: OUT_U13 -> OUT_U18
- U53 pad 18: OUT_U37 -> OUT_U19
- U53 pad 19: OUT_U25 -> OUT_U20
- U53 pad 2: OUT_U26 -> OUT_U23
- U53 pad 20: OUT_U12 -> OUT_U42
- U53 pad 21: OUT_U36 -> OUT_U44
- U53 pad 22: OUT_U24 -> OUT_U43
- U53 pad 23: OUT_U35 -> OUT_U30
- U53 pad 3: OUT_U38 -> OUT_U33
- U53 pad 4: OUT_U27 -> OUT_U22
- U53 pad 5: OUT_U39 -> OUT_U32
- U53 pad 6: OUT_U15 -> OUT_U41
- U53 pad 7: OUT_U28 -> OUT_U21
- U53 pad 8: OUT_U16 -> OUT_U40
- U53 pad 9: OUT_U17 -> OUT_U31
Routing:
- net OUT_U1: track 222.9 -> 33.2 mm
- net OUT_U11: track 71.5 -> 248.4 mm, vias 4 -> 2
- net OUT_U2: track 205.1 -> 52.8 mm, vias 4 -> 2
- net OUT_U6: track 280.8 -> 141.9 mm, vias 8 -> 2
- net OUT_U44: track 46.8 -> 184.1 mm, vias 4 -> 12
- net OUT_U5: track 256.7 -> 119.6 mm, vias 7 -> 2
- net OUT_U10: track 86.3 -> 219.4 mm
- net OUT_U3: track 188.6 -> 72.3 mm, vias 8 -> 2
- net OUT_U9: track 102.9 -> 207.7 mm, vias 6 -> 2
- net OUT_U43: track 76.1 -> 171.7 mm, vias 6 -> 10
- net OUT_U8: track 103.9 -> 186.8 mm, vias 10 -> 2
- net OUT_U4: track 165.2 -> 91.9 mm
- net LED_G_DRV: track 78.9 -> 13.3 mm, vias 3 -> 1
- net LED_R_DRV: track 70.2 -> 11.9 mm, vias 2 -> 1
- net OUT_U7: track 107.5 -> 164.3 mm
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Other:
- board size 267 x 88.2 mm -> 267 x 97.2 mm
- board text added: "< USB + jack - Teensy 4.0 on Audio Board Rev D"
- board text added: "eTuttino v0.5 HE"
- board text added: "eTuttino v0.5 HE - C-griff G3-E6 - beatconfused.com/etutti"
- board text removed: "Teensy 4.0 on Audio Board Rev D - USB + jack >"
- board text removed: "eTuttino v0.4 HE"
- board text removed: "eTuttino v0.4 HE - C-griff G3-E6 - beatconfused.com/etutti"

Commit message: eTuttino board v0.6 for the v7 case: hex grid 18.5, case outline, J3
- generate.py reads case/out/pcb_envelope.json: keys on the 18.5 mm
  hexagonal grid (rows 16.02 apart), the board outline (case cavity - 0.5,
  notched round the screw bosses), the bottom-plate pillars, the stack
  position from fit_check.py; ROWS, notes and firmware semantics unchanged
- build_pcb.py routes inside the outline polygon; the power LED moved to
  the controls board: R1/R2 stay, J3 (JST PH 8) carries 3.3 V, GND, pot
  (22), encoder A/B/SW (17/9/6), LED R/G; fails if a back-side part sits
  on a pillar; route order OUT_U41,OUT_U42,GND,LED_R,LED_G_DRV,OUT_U34
- result: DRC 0 errors / 0 warnings / 0 unconnected, firmware 44/44;
  KEY_INPUT rewritten in the sketch (compiles)
- case: pillar_points had rows 2-3 wrong (5.3 mm from a sensor); now one
  per three-key triangle (64): worst sag 0.044 mm at 3 N (was 0.37);
  envelope outlines now notched; FIT_CHECK lists what the board asks of
  the case
- mechanics.py checks the v7 board on those pillars; the #78 FreeCAD case
  (case.py, case_check.py, fab/etuttino_case_*) is removed; --renders off
  until the manuals are redone

Co-Authored-By: Claude Opus 5.5 <noreply@anthropic.com>
Parts:
- removed D1: LED 3mm red/green CC, LED_D3.0mm-3
- removed H1, H10, H11, H2, H3, H4, H5, H6, H7, H8, H9: MountingHole_2.2mm_M2, MountingHole_2.2mm_M2
- added J3: controls board, JST_PH_B8B-PH-K_1x08_P2.00mm_Vertical, F.Cu at (26.0, 48.3)
- moved C72 75.4 mm to (155.6, 12.7)
- moved U52 75.4 mm to (145.6, 12.7)
- moved C71 60.3 mm to (79.7, 85.8)
- moved U51 60.3 mm to (77.2, 76.0)
- moved C1 53.1 mm to (104.0, 71.0)
- moved SW1 53.1 mm to (104.0, 74.0)
- moved U1 53.1 mm to (104.0, 74.0)
- moved C12 53.0 mm to (94.8, 55.0)
- moved SW12 53.0 mm to (94.8, 58.0)
- moved U12 53.0 mm to (94.8, 58.0)
- moved C24 52.6 mm to (104.0, 39.0)
- moved SW24 52.6 mm to (104.0, 42.0)
- moved U24 52.6 mm to (104.0, 42.0)
- moved C2 52.6 mm to (122.5, 71.0)
- moved SW2 52.6 mm to (122.5, 74.0)
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Connections:
- J1 pad 11: (no net) -> ENC_B
- J1 pad 8: (no net) -> ENC_SW
- J2 pad 10: (no net) -> ENC_A
- J2 pad 5: (no net) -> POT
- U51 pad 19: OUT_U15 -> OUT_U1
- U51 pad 20: OUT_U4 -> OUT_U2
- U51 pad 22: OUT_U2 -> OUT_U4
- U51 pad 23: OUT_U1 -> OUT_U15
- U51 pad 7: OUT_U11 -> OUT_U10
- U51 pad 8: OUT_U10 -> OUT_U11
- U52 pad 16: (no net) -> OUT_U39
- U52 pad 17: (no net) -> OUT_U17
- U52 pad 18: (no net) -> OUT_U27
- U52 pad 19: OUT_U17 -> OUT_U36
- U52 pad 2: OUT_U39 -> OUT_U35
- U52 pad 20: (no net) -> OUT_U26
- U52 pad 21: OUT_U27 -> OUT_U38
- U52 pad 22: OUT_U28 -> OUT_U25
- U52 pad 23: OUT_U29 -> OUT_U24
- U52 pad 3: OUT_U38 -> OUT_U37
- U52 pad 4: OUT_U26 -> (no net)
- U52 pad 5: OUT_U24 -> (no net)
- U52 pad 6: OUT_U37 -> (no net)
- U52 pad 7: OUT_U25 -> OUT_U28
- U52 pad 8: OUT_U36 -> OUT_U29
- U52 pad 9: OUT_U35 -> (no net)
- U53 pad 16: OUT_U34 -> OUT_U42
- U53 pad 17: OUT_U18 -> OUT_U23
- U53 pad 18: OUT_U19 -> OUT_U22
- U53 pad 19: OUT_U20 -> OUT_U33
- U53 pad 2: OUT_U23 -> OUT_U30
- U53 pad 20: OUT_U42 -> OUT_U21
- U53 pad 21: OUT_U44 -> OUT_U19
- U53 pad 22: OUT_U43 -> OUT_U18
- U53 pad 23: OUT_U30 -> OUT_U41
- U53 pad 3: OUT_U33 -> OUT_U20
- U53 pad 4: OUT_U22 -> OUT_U40
- U53 pad 6: OUT_U41 -> OUT_U31
- U53 pad 7: OUT_U21 -> OUT_U43
- U53 pad 8: OUT_U40 -> OUT_U44
- U53 pad 9: OUT_U31 -> OUT_U34
Routing:
- net OUT_U43: track 171.7 -> 35.2 mm, vias 10 -> 2
- net OUT_U44: track 184.1 -> 52.3 mm, vias 12 -> 4
- net OUT_U41: track 114.3 -> 15.0 mm, vias 8 -> 2
- net OUT_U42: track 110.7 -> 13.2 mm, vias 10 -> 2
- net OUT_U36: track 90.0 -> 19.7 mm, vias 6 -> 2
- net OUT_U40: track 104.7 -> 39.1 mm, vias 6 -> 2
- net OUT_U39: track 114.8 -> 54.9 mm
- net OUT_U27: track 92.7 -> 33.8 mm
- net OUT_U38: track 102.7 -> 47.1 mm, vias 4 -> 6
- net ENC_A: track 0.00 -> 53.6 mm, vias 0 -> 2
- net OUT_U18: track 106.9 -> 55.0 mm
- net OUT_U26: track 81.8 -> 30.3 mm, vias 4 -> 6
- net COM1: track 37.2 -> 88.4 mm
- net OUT_U28: track 105.0 -> 53.8 mm, vias 4 -> 2
- net OUT_U30: track 92.8 -> 44.1 mm, vias 4 -> 2
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Other:
- board size 267 x 97.2 mm -> 321.8 x 91 mm
- board text added: "< USB - Teensy 4.0 on Audio Board Rev D"
- board text added: "controls board"
- board text added: "eTuttino v0.6 HE"
- board text added: "eTuttino v0.6 HE - C-griff G3-E6 - beatconfused.com/etutti"
- board text removed: "< USB + jack - Teensy 4.0 on Audio Board Rev D"
- board text removed: "POWER"
- board text removed: "eTuttino v0.5 HE"
- board text removed: "eTuttino v0.5 HE - C-griff G3-E6 - beatconfused.com/etutti"

Commit message: eTuttino v8: M2 board screws, 1.6 mm plate, controls board, firmware knobs
Implements case SPEC v8 (PR #88):
- case: 1.6 mm FR-4 plate (key tops z 26.6); two M2 screws from below
  through thicker pillars (30;60) and (12;70) with counterbores; two
  posts under the interface lid for the controls board; exports both in
  the PCB envelope
- main board v0.7: holes H1/H2 with a 3.5 mm copper-free ring, plate
  Gerbers at 1.6 mm; DRC 0/0/0, firmware 44/44, KEY_INPUT unchanged
- controls_pcb.py: the controls board (RK09K volume pot, EC11E encoder
  with switch, 3 mm red/green LED, vertical JST PH facing down to J3),
  routed with build_pcb's router; DRC 0/0/0
- firmware: pot (22) sets the volume and sends CC 7 back, ignored when no
  pot is detected at boot (checked on the real Teensy); encoder (17/9)
  steps the instrument and sends CC 25; its button confirms (saved to
  EEPROM) or returns to the default sound; LED blinks green while pending
- fit_check: the real controls board, its JST and cable, the M2 nuts;
  the side-entry JST hit the Chorus speaker, so it is a vertical one now

Co-Authored-By: Claude Opus 5.5 <noreply@anthropic.com>
Parts:
- added H1: MountingHole_2.2mm_M2, MountingHole_2.2mm_M2, F.Cu at (30.0, 60.0)
- added H2: MountingHole_2.2mm_M2, MountingHole_2.2mm_M2, F.Cu at (12.0, 70.0)
Other:
- board text added: "eTuttino v0.7 HE"
- board text added: "eTuttino v0.7 HE - C-griff G3-E6 - beatconfused.com/etutti"
- board text removed: "eTuttino v0.6 HE"
- board text removed: "eTuttino v0.6 HE - C-griff G3-E6 - beatconfused.com/etutti"
