File: etutti/hardware/pocket/pcb/kicad/pocket.kicad_pcb (KiCad board)
At the start: 4 copper layers, 242.2 x 94 mm, 146 parts, among them J1 PinSocket_1x14_P2.54mm_Vertic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, J2 PinSocket_1x14_P2.54mm_Vertic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, Q20 AO3401A, Q21 AO3400A, Q30 AO3401A, SW1 Gateron_Magnetic_MX_1u, SW10 Gateron_Magnetic_MX_1u, SW11 Gateron_Magnetic_MX_1u, SW12 Gateron_Magnetic_MX_1u, SW13 Gateron_Magnetic_MX_1u, SW14 Gateron_Magnetic_MX_1u, SW15 Gateron_Magnetic_MX_1u, SW16 Gateron_Magnetic_MX_1u, SW17 Gateron_Magnetic_MX_1u, SW18 Gateron_Magnetic_MX_1u, SW19 Gateron_Magnetic_MX_1u, SW2 Gateron_Magnetic_MX_1u, SW20 Gateron_Magnetic_MX_1u, SW21 Gateron_Magnetic_MX_1u, SW22 Gateron_Magnetic_MX_1u, SW23 Gateron_Magnetic_MX_1u, SW24 Gateron_Magnetic_MX_1u, SW25 Gateron_Magnetic_MX_1u, SW26 Gateron_Magnetic_MX_1u, SW27 Gateron_Magnetic_MX_1u, SW28 Gateron_Magnetic_MX_1u, SW3 Gateron_Magnetic_MX_1u, SW4 Gateron_Magnetic_MX_1u, SW5 Gateron_Magnetic_MX_1u, SW6 Gateron_Magnetic_MX_1u, SW7 Gateron_Magnetic_MX_1u, SW8 Gateron_Magnetic_MX_1u, SW9 Gateron_Magnetic_MX_1u, U1 TMAG5253BA3IQDMRR, U10 TMAG5253BA3IQDMRR, U11 TMAG5253BA3IQDMRR, U12 TMAG5253BA3IQDMRR, U13 TMAG5253BA3IQDMRR, U14 TMAG5253BA3IQDMRR, U15 TMAG5253BA3IQDMRR, U16 TMAG5253BA3IQDMRR, U17 TMAG5253BA3IQDMRR, U18 TMAG5253BA3IQDMRR, U19 TMAG5253BA3IQDMRR, U2 TMAG5253BA3IQDMRR, U20 TMAG5253BA3IQDMRR, U21 TMAG5253BA3IQDMRR, U22 TMAG5253BA3IQDMRR, U23 TMAG5253BA3IQDMRR, U24 TMAG5253BA3IQDMRR, U25 TMAG5253BA3IQDMRR, U26 TMAG5253BA3IQDMRR, U27 TMAG5253BA3IQDMRR, U28 TMAG5253BA3IQDMRR, U3 TMAG5253BA3IQDMRR, U4 TMAG5253BA3IQDMRR, U5 TMAG5253BA3IQDMRR, U51 CD74HC4067M96, U52 CD74HC4067M96, U53 74LVC1G04, U54 74LVC1G08, U55 74LVC1G08, U6 TMAG5253BA3IQDMRR, U60 BQ24074RGTR, U61 TPS63001DRCR, U62 PAM8302AASCR, U7 TMAG5253BA3IQDMRR, U8 TMAG5253BA3IQDMRR, U9 TMAG5253BA3IQDMRR

Commit message: eTuttino Pocket SPEC v4: F1 case finish + F2 boards closed, kit BOM
Co-Authored-By: Claude Opus 5.5 <noreply@anthropic.com>
Parts:
- added Q22: AO3400A, SOT-23, B.Cu at (90.6, 31.0)
- added Q31: AO3400A, SOT-23, B.Cu at (46.5, 20.6)
- added R26: 100k, R_0805_2012Metric, B.Cu at (94.4, 31.0)
Connections:
- U52 pad 6: OUT_U4 -> OUT_U16
- U52 pad 7: OUT_U16 -> OUT_U3
- U52 pad 8: OUT_U3 -> OUT_U4
Routing:
- net HP_VGND: track 45.6 -> 148.7 mm, vias 2 -> 5
- net OUT_U24: track 214.9 -> 135.2 mm, vias 9 -> 13
- net HP_R: track 42.3 -> 112.4 mm, vias 2 -> 7
- net LED_R: track 63.9 -> 109.3 mm, vias 7 -> 5
- net LED_G: track 22.7 -> 51.1 mm, vias 1 -> 3
- net VBUS: track 95.1 -> 121.2 mm, vias 4 -> 8
- net ENC_SW: track 33.7 -> 13.9 mm
- net SEL1: track 159.7 -> 177.8 mm, vias 4 -> 5
- net ENC_A: track 23.8 -> 39.5 mm
- net LEDR_A: track 27.7 -> 12.9 mm, vias 4 -> 2
- net OUT_U23: track 99.2 -> 86.4 mm, vias 12 -> 10
- net SEL0: track 162.5 -> 175.1 mm, vias 1 -> 5
- net PWR_A: track 33.8 -> 21.9 mm, vias 7 -> 1
- net QSG: track 6.83 -> 16.5 mm
- net LED_R_DRV: track 46.7 -> 38.3 mm, vias 3 -> 0
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Other:
- outline, holes or cut-outs redrawn
- board text added: "eTuttino Pocket v0.2"
- board text added: "eTuttino Pocket v0.2 - TMAG5253 on this side"
- board text removed: "eTuttino Pocket v0.1"
- board text removed: "eTuttino Pocket v0.1 - TMAG5253 on this side"

Commit message: eTuttino Pocket SPEC v5: F3 case for panel micro-USB/jack, knob recesses + F4 boards (FPC extension, VIN switch, no panel board)
Co-Authored-By: Claude Opus 5.5 <noreply@anthropic.com>
Parts:
- removed J_PNL: panel board, JST_SH_BM08B-SRSS-TB_1x08-1MP_P1.00mm_Vertical
- added D60: SMF5.0A, D_SOD-123F, B.Cu at (68.6, 8.00)
- added D61: B5819W, D_SOD-123, B.Cu at (34.8, 6.60)
- added J_JACK: wires from the panel jack (T, R, S, tip switch), PinHeader_1x04_P2.54mm_Vertical, F.Cu at (18.5, 28.6)
- added J_VBUS: VBUS wire from the Teensy's VUSB pad, SolderWire-0.25sqmm_1x01_D0.65mm_OD1.7mm, F.Cu at (18.5, 18.0)
- added Q23: AO3401A, SOT-23, B.Cu at (31.2, 6.00)
- added Q24: AO3400A, SOT-23, B.Cu at (92.8, 25.0)
- added R27: 100k, R_0805_2012Metric, B.Cu at (37.4, 10.4)
Connections:
- J2 pad 1: (no net) -> VIN_T
- U52 pad 17: OUT_U23 -> (no net)
- U52 pad 19: OUT_U24 -> OUT_U23
- U52 pad 20: (no net) -> OUT_U24
- U52 pad 6: OUT_U16 -> OUT_U4
- U52 pad 7: OUT_U3 -> OUT_U16
- U52 pad 8: OUT_U4 -> OUT_U3
Routing:
- net OUT_U23: track 86.4 -> 210.9 mm
- net QVG: track 0.00 -> 81.4 mm, vias 0 -> 2
- net OUT_U24: track 135.2 -> 216.1 mm, vias 13 -> 11
- net COM0: track 137.1 -> 188.9 mm
- net OUT_U10: track 112.0 -> 89.1 mm
- net COM1: track 79.0 -> 93.6 mm, vias 2 -> 3
- net SEL1: track 177.8 -> 191.6 mm, vias 5 -> 4
- net SEL0: track 175.1 -> 162.7 mm, vias 5 -> 2
- net OUT_U26: track 130.4 -> 140.4 mm, vias 10 -> 8
- net VIN_T: track 0.00 -> 8.12 mm, vias 0 -> 2
- net OUT_U21: track 77.4 -> 85.0 mm, vias 6 -> 4
- net HP_VGND: track 148.7 -> 156.2 mm, vias 5 -> 3
- net OUT_U27: track 129.3 -> 136.2 mm
- net VBUS: track 121.2 -> 128.0 mm, vias 8 -> 9
- net HP_TIPSW: track 29.8 -> 36.0 mm, vias 1 -> 4
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Other:
- board text added: "eTuttino Pocket v0.3"
- board text added: "eTuttino Pocket v0.3 - TMAG5253 on this side"
- board text removed: "eTuttino Pocket v0.2"
- board text removed: "eTuttino Pocket v0.2 - TMAG5253 on this side"
