File: etutti/hardware/pocket/pcb/kicad/pocket_controls.kicad_pcb (KiCad board)
At the start: 2 copper layers, 27.4 x 17.5 mm, 15 parts, among them SW1 EC11E 15/15

Commit message: eTuttino Pocket SPEC v4: F1 case finish + F2 boards closed, kit BOM
Co-Authored-By: Claude Opus 5.5 <noreply@anthropic.com>
Other:
- board text added: "CTL v0.2"
- board text removed: "CTL v0.1"
