File: etutti/hardware/pocket/pcb/kicad/pocket_pot.kicad_pcb (KiCad board)
At the start: 2 copper layers, 12 x 16 mm, 12 parts

Commit message: eTuttino Pocket SPEC v4: M1 assembly manual, volume board v0.2 (un-mirrored)
Co-Authored-By: Claude Opus 5.5 <noreply@anthropic.com>
Parts:
- moved JP1 10.0 mm to (1.00, 14.8)
- moved JP6 10.0 mm to (11.0, 14.8)
- moved JP2 7.60 mm to (2.20, 14.8)
- moved JP5 7.60 mm to (9.80, 14.8)
- moved JP3 5.20 mm to (3.40, 14.8)
- moved JP4 5.20 mm to (8.60, 14.8)
Routing:
- net GND: track 14.1 -> 14.9 mm
Other:
- board text added: "VOL v0.2"
- board text removed: "VOL"
