File: etutti/hardware/viaggio/pcb/kicad/viaggio.kicad_sch (KiCad schematic)
At the start: 0 parts

Commit message: eTutti Viaggio SPEC v2.1 step 3.2: placed board handed off for manual routing
- VE2a: power switch on the volume click (I1); flash W25Q64JVSSIM; both
  encoders EC11E18244A5 (the 15/15 has no stock); F2 = PJ-327A 5JJ (the
  PJ-313D-6A has no tip switch); PINOS.md and BOM updated. ERC 0/0, netlist
  check OK.
- VE2b: footprints.py writes viaggio.pretty (BGA-196 12x12 P0.8 from NXP
  figure 54, checked against rt1062_balls.json; jack; LED 1615; Gateron).
- VE2c: build_board.py builds the 246.5 x 95 board (R5 corners, M2 holes,
  silkscreen, JLC04121H-7628 stack-up, net classes, USB 90 ohm = 0.24/0.15
  per impedance.py) and places every part from viaggio_rev2.json.
- Routing: the own grid router could not close sector P (18 DRC errors),
  so J routes the board in KiCad with Freerouting. handoff_freerouting.py
  strips the tracks, links the board to the schematic, fixes 4 courtyard
  overlaps, makes In1/In2 plane layers and exports build/viaggio.dsn:
  DRC 0 errors, parity 0, 499 connections to route. Guide: ROTEAMENTO.md.

Co-Authored-By: Claude Opus 5.5 <noreply@anthropic.com>
Other:
- note added: "Placa: pcb/build_board.py (posicionamento + setor P). Ligacoes entre folhas por rotulos globais."
- note added: "eTutti Viaggio · esquema eletrico (SPEC v2.1, passo 3.2). Uma folha por setor da SPEC (secao 3)."
- note removed: "Sem placa: nada posicionado nem roteado neste passo. Ligacoes entre folhas por rotulos globais."
- note removed: "eTutti Viaggio · esquema eletrico (SPEC v2, passo 3.1). Uma folha por setor da SPEC (secao 3)."
Changed lines of the file:
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@@
 	(generator_version "10.0")
 	(paper "A4")
-	(title_block (title "eTutti Viaggio · esquema") (date "2026-10-24") (rev "SPEC v2 - passo 3.1") (company "beatconfused.com") (comment 1 "etutti/hardware/viaggio/pcb/schematic.py escreve este arquivo; nao editar a mao"))
-	(text "eTutti Viaggio · esquema eletrico (SPEC v2, passo 3.1). Uma folha por setor da SPEC (secao 3)." (exclude_from_sim no) (at 25 15 0) (effects (font (size 2 2)) (justify left)))
+	(title_block (title "eTutti Viaggio · esquema") (date "2026-10-24") (rev "SPEC v2.1 - passo 3.2") (company "beatconfused.com") (comment 1 "etutti/hardware/viaggio/pcb/schematic.py escreve este arquivo; nao editar a mao"))
+	(text "eTutti Viaggio · esquema eletrico (SPEC v2.1, passo 3.2). Uma folha por setor da SPEC (secao 3)." (exclude_from_sim no) (at 25 15 0) (effects (font (size 2 2)) (justify left)))
 	(text "Campo 'Codigo' = codigo da peca na SPEC (P1...T4), o mesmo de concept/rev2/out/viaggio_rev2.json." (exclude_from_sim no) (at 25 21 0) (effects (font (size 2 2)) (justify left)))
-	(text "Sem placa: nada posicionado nem roteado neste passo. Ligacoes entre folhas por rotulos globais." (exclude_from_sim no) (at 25 27 0) (effects (font (size 2 2)) (justify left)))
+	(text "Placa: pcb/build_board.py (posicionamento + setor P). Ligacoes entre folhas por rotulos globais." (exclude_from_sim no) (at 25 27 0) (effects (font (size 2 2)) (justify left)))
 	(text "PWR_FLAG abaixo: redes alimentadas por conector, ferrite, indutor ou diodo (o ERC nao ve a fonte)." (exclude_from_sim no) (at 25 33 0) (effects (font (size 2 2)) (justify left)))
 	(sheet (at 25 45) (size 70 25) (exclude_from_sim no) (in_bom yes) (on_board yes) (dnp no) (fields_autoplaced yes) (stroke (width 0.1524) (type solid)) (fill (color 0 0 0 0.0000))
