File: etutti/hardware/viaggio/pcb/kicad/viaggio_E.kicad_sch (KiCad schematic)
At the start: 45 parts, among them J201 TYPE-C-31-M-12, J202 S3B-PH-SM4-TB, Q201 AO3401A, Q202 AO3400A, Q203 AO3401A, U201 USBLC6-2SC6, U202 BQ24074RGTR, U203 74LVC1G08, U204 TPS63001DRCR, U205 XC6206P332MR, U206 74LVC1G08

Commit message: eTutti Viaggio SPEC v2.1 step 3.2: placed board handed off for manual routing
- VE2a: power switch on the volume click (I1); flash W25Q64JVSSIM; both
  encoders EC11E18244A5 (the 15/15 has no stock); F2 = PJ-327A 5JJ (the
  PJ-313D-6A has no tip switch); PINOS.md and BOM updated. ERC 0/0, netlist
  check OK.
- VE2b: footprints.py writes viaggio.pretty (BGA-196 12x12 P0.8 from NXP
  figure 54, checked against rt1062_balls.json; jack; LED 1615; Gateron).
- VE2c: build_board.py builds the 246.5 x 95 board (R5 corners, M2 holes,
  silkscreen, JLC04121H-7628 stack-up, net classes, USB 90 ohm = 0.24/0.15
  per impedance.py) and places every part from viaggio_rev2.json.
- Routing: the own grid router could not close sector P (18 DRC errors),
  so J routes the board in KiCad with Freerouting. handoff_freerouting.py
  strips the tracks, links the board to the schematic, fixes 4 courtyard
  overlaps, makes In1/In2 plane layers and exports build/viaggio.dsn:
  DRC 0 errors, parity 0, 499 connections to route. Guide: ROTEAMENTO.md.

Co-Authored-By: Claude Opus 5.5 <noreply@anthropic.com>
Connections:
- net SEL_SW renamed VOL_SW
- net SEL_SW_N renamed VOL_SW_N
Other:
- note added: "EN do TPS63001 = PMIC_ON_REQ E (clique do volume OU KEEP OU USB com o aparelho ligado)."
- note removed: "EN do TPS63001 = PMIC_ON_REQ E (clique do seletor OU KEEP OU USB com o aparelho ligado)."
Changed lines of the file:
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@@
 	(generator_version "10.0")
 	(paper "A2")
-	(title_block (title "eTutti Viaggio · E · Energia") (date "2026-10-24") (rev "SPEC v2 - passo 3.1") (company "beatconfused.com") (comment 1 "etutti/hardware/viaggio/pcb/schematic.py escreve este arquivo; nao editar a mao"))
+	(title_block (title "eTutti Viaggio · E · Energia") (date "2026-10-24") (rev "SPEC v2.1 - passo 3.2") (company "beatconfused.com") (comment 1 "etutti/hardware/viaggio/pcb/schematic.py escreve este arquivo; nao editar a mao"))
 	(text "E · Energia: USB-C -> BQ24074 (USB500, 500 mA, NTC) -> VSYS -> TPS63001 (3,3 V)." (exclude_from_sim no) (at 15 18 0) (effects (font (size 2 2)) (justify left)))
-	(text "EN do TPS63001 = PMIC_ON_REQ E (clique do seletor OU KEEP OU USB com o aparelho ligado)." (exclude_from_sim no) (at 15 23 0) (effects (font (size 2 2)) (justify left)))
+	(text "EN do TPS63001 = PMIC_ON_REQ E (clique do volume OU KEEP OU USB com o aparelho ligado)." (exclude_from_sim no) (at 15 23 0) (effects (font (size 2 2)) (justify left)))
 	(text "E5: LDO sempre ligado para o SNVS. Luz de carga so com o aparelho desligado (Q202)." (exclude_from_sim no) (at 15 28 0) (effects (font (size 2 2)) (justify left)))
 	(symbol (lib_id "viaggio:USB_C_Receptacle_USB2.0_16P") (at 25.4 63.5 0) (unit 1) (exclude_from_sim no) (in_bom yes) (on_board yes) (dnp no)
@@
 		(property "Footprint" "Package_TO_SOT_SMD:SOT-23" (at 177.8 124.46 0) (hide yes) (effects (font (size 1.27 1.27))))
 		(property "Datasheet" "https://www.aosmd.com/res/datasheets/AO3401A.pdf" (at 177.8 124.46 0) (hide yes) (effects (font (size 1.27 1.27))))
-		(property "Description" "o clique do seletor liga o EN" (at 177.8 124.46 0) (hide yes) (effects (font (size 1.27 1.27))))
+		(property "Description" "o clique do volume liga o EN" (at 177.8 124.46 0) (hide yes) (effects (font (size 1.27 1.27))))
 		(property "Codigo" "E3" (at 180.34 115.57 0) (effects (font (size 1.27 1.27)) (justify right)))
 		(property "LCSC" "C15127" (at 177.8 124.46 0) (hide yes) (effects (font (size 1.27 1.27))))
@@
 	)
 	(wire (pts (xy 172.72 124.46) (xy 170.18 124.46)) (stroke (width 0) (type default)))
-	(global_label "SEL_SW_N" (shape passive) (at 170.18 124.46 180) (fields_autoplaced yes) (effects (font (size 1.27 1.27)) (justify right)) (property "Intersheetrefs" "${INTERSHEET_REFS}" (at 170.18 124.46 0) (hide yes) (effects (font (size 1.27 1.27)) (justify right))))
+	(global_label "VOL_SW_N" (shape passive) (at 170.18 124.46 180) (fields_autoplaced yes) (effects (font (size 1.27 1.27)) (justify right)) (property "Intersheetrefs" "${INTERSHEET_REFS}" (at 170.18 124.46 0) (hide yes) (effects (font (size 1.27 1.27)) (justify right))))
 	(wire (pts (xy 180.34 129.54) (xy 180.34 132.08)) (stroke (width 0) (type default)))
 	(global_label "VSYS" (shape passive) (at 180.34 132.08 270) (fields_autoplaced yes) (effects (font (size 1.27 1.27)) (justify right)) (property "Intersheetrefs" "${INTERSHEET_REFS}" (at 180.34 132.08 0) (hide yes) (effects (font (size 1.27 1.27)) (justify right))))
@@
 	(global_label "VSYS" (shape passive) (at 194.31 109.22 180) (fields_autoplaced yes) (effects (font (size 1.27 1.27)) (justify right)) (property "Intersheetrefs" "${INTERSHEET_REFS}" (at 194.31 109.22 0) (hide yes) (effects (font (size 1.27 1.27)) (justify right))))
 	(wire (pts (xy 204.47 109.22) (xy 207.01 109.22)) (stroke (width 0) (type default)))
-	(global_label "SEL_SW_N" (shape passive) (at 207.01 109.22 0) (fields_autoplaced yes) (effects (font (size 1.27 1.27)) (justify left)) (property "Intersheetrefs" "${INTERSHEET_REFS}" (at 207.01 109.22 0) (hide yes) (effects (font (size 1.27 1.27)) (justify left))))
+	(global_label "VOL_SW_N" (shape passive) (at 207.01 109.22 0) (fields_autoplaced yes) (effects (font (size 1.27 1.27)) (justify left)) (property "Intersheetrefs" "${INTERSHEET_REFS}" (at 207.01 109.22 0) (hide yes) (effects (font (size 1.27 1.27)) (justify left))))
 	(symbol (lib_id "viaggio:R") (at 241.3 109.22 90) (unit 1) (exclude_from_sim no) (in_bom yes) (on_board yes) (dnp no)
 		(property "Reference" "R211" (at 237.49 105.41 0) (effects (font (size 1.27 1.27)) (justify left)))
@@
 		(property "Footprint" "Package_TO_SOT_SMD:SOT-23" (at 35.56 157.48 0) (hide yes) (effects (font (size 1.27 1.27))))
 		(property "Datasheet" "https://www.diodes.com/assets/Datasheets/ds11005.pdf" (at 35.56 157.48 0) (hide yes) (effects (font (size 1.27 1.27))))
-		(property "Description" "o clique chega ao pino 6 e ao ONOFF do SNVS sem levar o VSYS a eles" (at 35.56 157.48 0) (hide yes) (effects (font (size 1.27 1.27))))
+		(property "Description" "o clique do volume chega ao pino 25 e ao ONOFF do SNVS sem levar o VSYS a eles" (at 35.56 157.48 0) (hide yes) (effects (font (size 1.27 1.27))))
 		(property "Codigo" "E3" (at 43.18 153.67 0) (effects (font (size 1.27 1.27)) (justify right)))
 		(property "LCSC" "C134405" (at 35.56 157.48 0) (hide yes) (effects (font (size 1.27 1.27))))
@@
 	)
 	(wire (pts (xy 27.94 157.48) (xy 25.4 157.48)) (stroke (width 0) (type default)))
-	(global_label "SEL_SW" (shape passive) (at 25.4 157.48 180) (fields_autoplaced yes) (effects (font (size 1.27 1.27)) (justify right)) (property "Intersheetrefs" "${INTERSHEET_REFS}" (at 25.4 157.48 0) (hide yes) (effects (font (size 1.27 1.27)) (justify right))))
+	(global_label "VOL_SW" (shape passive) (at 25.4 157.48 180) (fields_autoplaced yes) (effects (font (size 1.27 1.27)) (justify right)) (property "Intersheetrefs" "${INTERSHEET_REFS}" (at 25.4 157.48 0) (hide yes) (effects (font (size 1.27 1.27)) (justify right))))
 	(wire (pts (xy 43.18 157.48) (xy 45.72 157.48)) (stroke (width 0) (type default)))
 	(global_label "ONOFF" (shape passive) (at 45.72 157.48 0) (fields_autoplaced yes) (effects (font (size 1.27 1.27)) (justify left)) (property "Intersheetrefs" "${INTERSHEET_REFS}" (at 45.72 157.48 0) (hide yes) (effects (font (size 1.27 1.27)) (justify left))))
 	(wire (pts (xy 35.56 162.56) (xy 35.56 165.1)) (stroke (width 0) (type default)))
-	(global_label "SEL_SW_N" (shape passive) (at 35.56 165.1 270) (fields_autoplaced yes) (effects (font (size 1.27 1.27)) (justify right)) (property "Intersheetrefs" "${INTERSHEET_REFS}" (at 35.56 165.1 0) (hide yes) (effects (font (size 1.27 1.27)) (justify right))))
+	(global_label "VOL_SW_N" (shape passive) (at 35.56 165.1 270) (fields_autoplaced yes) (effects (font (size 1.27 1.27)) (justify right)) (property "Intersheetrefs" "${INTERSHEET_REFS}" (at 35.56 165.1 0) (hide yes) (effects (font (size 1.27 1.27)) (justify right))))
 	(symbol (lib_id "viaggio:TPS63001") (at 83.82 167.64 0) (unit 1) (exclude_from_sim no) (in_bom yes) (on_board yes) (dnp no)
 		(property "Reference" "U204" (at 73.66 153.67 0) (effects (font (size 1.27 1.27)) (justify left)))
