File: etutti/hardware/viaggio/pcb/kicad/viaggio_I.kicad_sch (KiCad schematic)
At the start: 7 parts, among them SW401 EC11E 15/15 com chave, SW402 EC11E 15/15 com chave, SW403 Program

Commit message: eTutti Viaggio SPEC v2.1 step 3.2: placed board handed off for manual routing
- VE2a: power switch on the volume click (I1); flash W25Q64JVSSIM; both
  encoders EC11E18244A5 (the 15/15 has no stock); F2 = PJ-327A 5JJ (the
  PJ-313D-6A has no tip switch); PINOS.md and BOM updated. ERC 0/0, netlist
  check OK.
- VE2b: footprints.py writes viaggio.pretty (BGA-196 12x12 P0.8 from NXP
  figure 54, checked against rt1062_balls.json; jack; LED 1615; Gateron).
- VE2c: build_board.py builds the 246.5 x 95 board (R5 corners, M2 holes,
  silkscreen, JLC04121H-7628 stack-up, net classes, USB 90 ohm = 0.24/0.15
  per impedance.py) and places every part from viaggio_rev2.json.
- Routing: the own grid router could not close sector P (18 DRC errors),
  so J routes the board in KiCad with Freerouting. handoff_freerouting.py
  strips the tracks, links the board to the schematic, fixes 4 courtyard
  overlaps, makes In1/In2 plane layers and exports build/viaggio.dsn:
  DRC 0 errors, parity 0, 499 connections to route. Guide: ROTEAMENTO.md.

Co-Authored-By: Claude Opus 5.5 <noreply@anthropic.com>
Parts:
- D401: footprint (none) -> viaggio:LED_1615_RG_4pad; symbol viaggio:LED_Dual_AAKK -> viaggio:LED_RG_1615
- SW401, SW402: value EC11E 15/15 com chave -> EC11E18244A5; LCSC (none) -> C255515
Connections:
- net GND: now also D401.2 (K1); no longer D401.3 (K1)
- net LED_G_A: now also D401.3 (A2); no longer D401.2 (A2)
- net SEL_SW_N renamed SEL_SW
- net VOL_SW renamed VOL_SW_N
Other:
- note added: "O clique do volume (I1) liga/desliga (circuito na folha E); o do seletor (I2) e uma entrada comum (pino 6)."
- note removed: "O clique do seletor vai ao GND; o liga/desliga esta na folha E."
- moved on the sheet: SW402
