File: etutti/hardware/viaggio/pcb/kicad/viaggio_P.kicad_sch (KiCad schematic)
At the start: 42 parts, among them U101 MIMXRT1062DVJ6B, U102 PJRC MKL02 bootloader (Teensy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, U103 W25Q64JVSSIQ, U104 APS6404L-3SQR-ZR, Y101 24MHz, Y102 32.768kHz

Commit message: eTutti Viaggio SPEC v2.1 step 3.2: placed board handed off for manual routing
- VE2a: power switch on the volume click (I1); flash W25Q64JVSSIM; both
  encoders EC11E18244A5 (the 15/15 has no stock); F2 = PJ-327A 5JJ (the
  PJ-313D-6A has no tip switch); PINOS.md and BOM updated. ERC 0/0, netlist
  check OK.
- VE2b: footprints.py writes viaggio.pretty (BGA-196 12x12 P0.8 from NXP
  figure 54, checked against rt1062_balls.json; jack; LED 1615; Gateron).
- VE2c: build_board.py builds the 246.5 x 95 board (R5 corners, M2 holes,
  silkscreen, JLC04121H-7628 stack-up, net classes, USB 90 ohm = 0.24/0.15
  per impedance.py) and places every part from viaggio_rev2.json.
- Routing: the own grid router could not close sector P (18 DRC errors),
  so J routes the board in KiCad with Freerouting. handoff_freerouting.py
  strips the tracks, links the board to the schematic, fixes 4 courtyard
  overlaps, makes In1/In2 plane layers and exports build/viaggio.dsn:
  DRC 0 errors, parity 0, 499 connections to route. Guide: ROTEAMENTO.md.

Co-Authored-By: Claude Opus 5.5 <noreply@anthropic.com>
Parts:
- C109, C112, C114: footprint Capacitor_SMD:C_0603_1608Metric -> Capacitor_SMD:C_0402_1005Metric; LCSC C19666 -> C23733
- C117: footprint Capacitor_SMD:C_0603_1608Metric -> Capacitor_SMD:C_0402_1005Metric; LCSC C19702 -> C15525
- U101: footprint (none) -> viaggio:BGA-196_12x12mm_P0.8mm_RT1062
- U103: value W25Q64JVSSIQ -> W25Q64JVSSIM; LCSC C179171 -> C5362615
