File: etutti/hardware/viaggio_micromod/pcb/kicad/viaggio_micromod.kicad_pcb (KiCad board)
At the start: 4 copper layers, 246.5 x 95 mm, 177 parts, among them J101 91302-42-067RCE, J201 TYPE-C-31-M-12, J202 S3B-PH-SM4-TB, J301 PJ-327A 5JJ, J501 alto-falante (fios), Q201 AO3401A, Q202 AO3400A, Q203 AO3401A, SW1 Gateron_Magnetic_MX_1u, SW10 Gateron_Magnetic_MX_1u, SW11 Gateron_Magnetic_MX_1u, SW12 Gateron_Magnetic_MX_1u, SW13 Gateron_Magnetic_MX_1u, SW14 Gateron_Magnetic_MX_1u, SW15 Gateron_Magnetic_MX_1u, SW16 Gateron_Magnetic_MX_1u, SW17 Gateron_Magnetic_MX_1u, SW18 Gateron_Magnetic_MX_1u, SW19 Gateron_Magnetic_MX_1u, SW2 Gateron_Magnetic_MX_1u, SW20 Gateron_Magnetic_MX_1u, SW21 Gateron_Magnetic_MX_1u, SW22 Gateron_Magnetic_MX_1u, SW23 Gateron_Magnetic_MX_1u, SW24 Gateron_Magnetic_MX_1u, SW25 Gateron_Magnetic_MX_1u, SW26 Gateron_Magnetic_MX_1u, SW27 Gateron_Magnetic_MX_1u, SW28 Gateron_Magnetic_MX_1u, SW3 Gateron_Magnetic_MX_1u, SW4 Gateron_Magnetic_MX_1u, SW401 EC11E18244A5, SW402 EC11E18244A5, SW403 Program, SW5 Gateron_Magnetic_MX_1u, SW6 Gateron_Magnetic_MX_1u, SW7 Gateron_Magnetic_MX_1u, SW8 Gateron_Magnetic_MX_1u, SW9 Gateron_Magnetic_MX_1u, U201 USBLC6-2SC6, U202 BQ24074RGTR, U203 74LVC1G08, U204 TPS63001DRCR, U301 SGTL5000XNLA3, U302 XC6206P182MR, U501 MAX98357AETE+T, U601 74HC4067PW, U602 74HC4067PW, U603 74LVC1G04, U604 74LVC1G08, U605 74LVC1G08, U701 TMAG5253BA3IQDMRR, U702 TMAG5253BA3IQDMRR, U703 TMAG5253BA3IQDMRR, U704 TMAG5253BA3IQDMRR, U705 TMAG5253BA3IQDMRR, U706 TMAG5253BA3IQDMRR, U707 TMAG5253BA3IQDMRR, U708 TMAG5253BA3IQDMRR, U709 TMAG5253BA3IQDMRR, U710 TMAG5253BA3IQDMRR, U711 TMAG5253BA3IQDMRR, U712 TMAG5253BA3IQDMRR, U713 TMAG5253BA3IQDMRR, U714 TMAG5253BA3IQDMRR, U715 TMAG5253BA3IQDMRR, U716 TMAG5253BA3IQDMRR, U717 TMAG5253BA3IQDMRR, U718 TMAG5253BA3IQDMRR, U719 TMAG5253BA3IQDMRR, U720 TMAG5253BA3IQDMRR, U721 TMAG5253BA3IQDMRR, U722 TMAG5253BA3IQDMRR, U723 TMAG5253BA3IQDMRR, U724 TMAG5253BA3IQDMRR, U725 TMAG5253BA3IQDMRR, U726 TMAG5253BA3IQDMRR, U727 TMAG5253BA3IQDMRR, U728 TMAG5253BA3IQDMRR

Commit message: eTutti Viaggio MicroMod: route only the USB pair (authorised exception)
route_usb.py (KiCad python, no router or path search) adds the USB_DP /
USB_DN tracks computed from the J201, U201 and J101 pads: F.Cu, 0.24 mm,
0.15 mm gap, 45 degree corners, one 0.5/0.3 via per net inside J101's
courtyard, B.Cu stubs to pads 3/5, all locked. It only splices the USB
items (and the In1 GND fill) into the PR #119 board.

DRC: 0 violations, parity 0, unconnected 431 -> 423 (USB 0 left).
USB_DP 32.90 mm, USB_DN 32.74 mm J201 -> J101 (34.87 / 35.50 with the
J201 joins), 1 via each. No other net routed.

Co-Authored-By: Claude Opus 5.5 <noreply@anthropic.com>
Routing:
- net USB_DN: track 0.00 -> 35.5 mm, vias 0 -> 1
- net USB_DP: track 0.00 -> 34.9 mm, vias 0 -> 1

Commit message: eTutti Viaggio MicroMod: U201 rotated 180 degrees, USB pair redone straight
- build_board.py: U201 (E2) rot 180 (D201 moved 0.015 mm with it); only
  the USB pair had been routed, so the board was rebuilt and re-routed.
- route_usb.py: straight J201 -> U201 -> J101 pair, no loop; a hook at
  J101 swaps the pair order and evens the lengths. USB_DP 21.50 mm,
  USB_DN 21.97 mm (delta 0.47), 1 via each, locked.
- D- join under the USB-C body stays in F.Cu: the HRO TYPE-C-31-M-12
  bottom shell ends ~0.3 mm before it (to be checked on a real part).
- DRC: 0 violations, parity 0, 423 unconnected (USB 0 left).
- ELETRONICA.md / ROTEAMENTO.md: where J puts the U201 GND/VBUS vias.

Co-Authored-By: Claude Opus 5.5 <noreply@anthropic.com>
Parts:
- turned U201 to 180 degrees
Routing:
- net USB_DP: track 34.9 -> 23.5 mm
- net USB_DN: track 35.5 -> 24.7 mm
