File: etutti/hardware/viaggio_j1/kicad/viaggio_micromod.kicad_pcb (KiCad board)
At the start: 4 copper layers, 246.5 x 95 mm, 177 parts, among them J101 91302-42-067RCE, J201 TYPE-C-31-M-12, J202 S3B-PH-SM4-TB, J301 PJ-327A 5JJ, J501 alto-falante (fios), Q201 AO3401A, Q202 AO3400A, Q203 AO3401A, SW1 Gateron_Magnetic_MX_1u, SW10 Gateron_Magnetic_MX_1u, SW11 Gateron_Magnetic_MX_1u, SW12 Gateron_Magnetic_MX_1u, SW13 Gateron_Magnetic_MX_1u, SW14 Gateron_Magnetic_MX_1u, SW15 Gateron_Magnetic_MX_1u, SW16 Gateron_Magnetic_MX_1u, SW17 Gateron_Magnetic_MX_1u, SW18 Gateron_Magnetic_MX_1u, SW19 Gateron_Magnetic_MX_1u, SW2 Gateron_Magnetic_MX_1u, SW20 Gateron_Magnetic_MX_1u, SW21 Gateron_Magnetic_MX_1u, SW22 Gateron_Magnetic_MX_1u, SW23 Gateron_Magnetic_MX_1u, SW24 Gateron_Magnetic_MX_1u, SW25 Gateron_Magnetic_MX_1u, SW26 Gateron_Magnetic_MX_1u, SW27 Gateron_Magnetic_MX_1u, SW28 Gateron_Magnetic_MX_1u, SW3 Gateron_Magnetic_MX_1u, SW4 Gateron_Magnetic_MX_1u, SW401 EC11E18244A5, SW402 EC11E18244A5, SW403 Program, SW5 Gateron_Magnetic_MX_1u, SW6 Gateron_Magnetic_MX_1u, SW7 Gateron_Magnetic_MX_1u, SW8 Gateron_Magnetic_MX_1u, SW9 Gateron_Magnetic_MX_1u, U201 USBLC6-2SC6, U202 BQ24074RGTR, U203 74LVC1G08, U204 TPS63001DRCR, U301 SGTL5000XNLA3, U302 XC6206P182MR, U501 MAX98357AETE+T, U601 74HC4067PW, U602 74HC4067PW, U603 74LVC1G04, U604 74LVC1G08, U605 74LVC1G08, U701 TMAG5253BA3IQDMRR, U702 TMAG5253BA3IQDMRR, U703 TMAG5253BA3IQDMRR, U704 TMAG5253BA3IQDMRR, U705 TMAG5253BA3IQDMRR, U706 TMAG5253BA3IQDMRR, U707 TMAG5253BA3IQDMRR, U708 TMAG5253BA3IQDMRR, U709 TMAG5253BA3IQDMRR, U710 TMAG5253BA3IQDMRR, U711 TMAG5253BA3IQDMRR, U712 TMAG5253BA3IQDMRR, U713 TMAG5253BA3IQDMRR, U714 TMAG5253BA3IQDMRR, U715 TMAG5253BA3IQDMRR, U716 TMAG5253BA3IQDMRR, U717 TMAG5253BA3IQDMRR, U718 TMAG5253BA3IQDMRR, U719 TMAG5253BA3IQDMRR, U720 TMAG5253BA3IQDMRR, U721 TMAG5253BA3IQDMRR, U722 TMAG5253BA3IQDMRR, U723 TMAG5253BA3IQDMRR, U724 TMAG5253BA3IQDMRR, U725 TMAG5253BA3IQDMRR, U726 TMAG5253BA3IQDMRR, U727 TMAG5253BA3IQDMRR, U728 TMAG5253BA3IQDMRR

Commit message: viaggio-j1-roteamento
Routing:
- net EN_A: track 0.00 -> 320.9 mm, vias 0 -> 15
- net EN_B: track 0.00 -> 277.2 mm, vias 0 -> 11
- net +3V3: track 0.00 -> 204.0 mm, vias 0 -> 4
- net MUX_S3: track 0.00 -> 185.0 mm, vias 0 -> 4
- net MUX_S1: track 0.00 -> 182.0 mm, vias 0 -> 4
- net MUX_S0: track 0.00 -> 179.1 mm, vias 0 -> 3
- net MUX_S2: track 0.00 -> 170.9 mm, vias 0 -> 4
- net MUX_R_COM: track 0.00 -> 167.3 mm, vias 0 -> 2
- net SENS_EN: track 0.00 -> 129.1 mm, vias 0 -> 2
- net MUX_L_COM: track 0.00 -> 99.4 mm, vias 0 -> 2
- net I2S_TX: track 0.00 -> 94.9 mm, vias 0 -> 4
- net I2S_LRCLK: track 0.00 -> 85.9 mm, vias 0 -> 3
- net I2S_BCLK: track 0.00 -> 85.2 mm, vias 0 -> 3
- net AMP_SD: track 0.00 -> 83.3 mm, vias 0 -> 2
- net OUT_K04: track 0.00 -> 81.2 mm, vias 0 -> 2
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