File: etutti/hardware/viaggio_j1/kicad/viaggio_micromod.kicad_pcb (KiCad board)
At the start: 4 copper layers, 246.5 x 95 mm, 177 parts, among them J101 91302-42-067RCE, J201 TYPE-C-31-M-12, J202 S3B-PH-SM4-TB, J301 PJ-327A 5JJ, J501 alto-falante (fios), Q201 AO3401A, Q202 AO3400A, Q203 AO3401A, SW1 Gateron_Magnetic_MX_1u, SW10 Gateron_Magnetic_MX_1u, SW11 Gateron_Magnetic_MX_1u, SW12 Gateron_Magnetic_MX_1u, SW13 Gateron_Magnetic_MX_1u, SW14 Gateron_Magnetic_MX_1u, SW15 Gateron_Magnetic_MX_1u, SW16 Gateron_Magnetic_MX_1u, SW17 Gateron_Magnetic_MX_1u, SW18 Gateron_Magnetic_MX_1u, SW19 Gateron_Magnetic_MX_1u, SW2 Gateron_Magnetic_MX_1u, SW20 Gateron_Magnetic_MX_1u, SW21 Gateron_Magnetic_MX_1u, SW22 Gateron_Magnetic_MX_1u, SW23 Gateron_Magnetic_MX_1u, SW24 Gateron_Magnetic_MX_1u, SW25 Gateron_Magnetic_MX_1u, SW26 Gateron_Magnetic_MX_1u, SW27 Gateron_Magnetic_MX_1u, SW28 Gateron_Magnetic_MX_1u, SW3 Gateron_Magnetic_MX_1u, SW4 Gateron_Magnetic_MX_1u, SW401 EC11E18244A5, SW402 EC11E18244A5, SW403 Program, SW5 Gateron_Magnetic_MX_1u, SW6 Gateron_Magnetic_MX_1u, SW7 Gateron_Magnetic_MX_1u, SW8 Gateron_Magnetic_MX_1u, SW9 Gateron_Magnetic_MX_1u, U201 USBLC6-2SC6, U202 BQ24074RGTR, U203 74LVC1G08, U204 TPS63001DRCR, U301 SGTL5000XNLA3, U302 XC6206P182MR, U501 MAX98357AETE+T, U601 74HC4067PW, U602 74HC4067PW, U603 74LVC1G04, U604 74LVC1G08, U605 74LVC1G08, U701 TMAG5253BA3IQDMRR, U702 TMAG5253BA3IQDMRR, U703 TMAG5253BA3IQDMRR, U704 TMAG5253BA3IQDMRR, U705 TMAG5253BA3IQDMRR, U706 TMAG5253BA3IQDMRR, U707 TMAG5253BA3IQDMRR, U708 TMAG5253BA3IQDMRR, U709 TMAG5253BA3IQDMRR, U710 TMAG5253BA3IQDMRR, U711 TMAG5253BA3IQDMRR, U712 TMAG5253BA3IQDMRR, U713 TMAG5253BA3IQDMRR, U714 TMAG5253BA3IQDMRR, U715 TMAG5253BA3IQDMRR, U716 TMAG5253BA3IQDMRR, U717 TMAG5253BA3IQDMRR, U718 TMAG5253BA3IQDMRR, U719 TMAG5253BA3IQDMRR, U720 TMAG5253BA3IQDMRR, U721 TMAG5253BA3IQDMRR, U722 TMAG5253BA3IQDMRR, U723 TMAG5253BA3IQDMRR, U724 TMAG5253BA3IQDMRR, U725 TMAG5253BA3IQDMRR, U726 TMAG5253BA3IQDMRR, U727 TMAG5253BA3IQDMRR, U728 TMAG5253BA3IQDMRR

Commit message: eTutti Viaggio J1 rota restante: lote 3 — I2C e +3V3 junto do J101
I2C_SDA and I2C_SCL closed (0.2 mm); 4 +3V3 links left of the keyboard.
The first I2C_SDA path cut J101.36 off the GND pour; the lot was redone
with that pin's copper protected. U301.21 and C304.2 (codec GND) left
out: J's In2 tracks run under the exposed pad, no via spot.
DRC: no new clearance/short/hole; unrouted 34 -> 28.

Co-Authored-By: Claude Opus 5.5 <noreply@anthropic.com>
Routing:
- net I2C_SDA: track 33.3 -> 45.9 mm
- net I2C_SCL: track 34.8 -> 44.6 mm, vias 4 -> 6
- net +3V3: track 245.1 -> 247.5 mm, vias 47 -> 51
Changed lines of the file:
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@@
 		(net "VBUS")
+	)
+	(segment
+		(start 25.500503 56.660365)
+		(end 24.750503 57.410365)
+		(width 0.3)
+		(layer "F.Cu")
+		(net "+3V3")
+	)
+	(via
+		(at 30.945214 23.935)
+		(size 0.5)
+		(drill 0.3)
+		(layers "F.Cu" "B.Cu")
+		(net "+3V3")
+	)
+	(via
+		(at 24.750503 57.410365)
+		(size 0.5)
+		(drill 0.3)
+		(layers "F.Cu" "B.Cu")
+		(net "+3V3")
+	)
+	(via
+		(at 25.500503 56.660365)
+		(size 0.5)
+		(drill 0.3)
+		(layers "F.Cu" "B.Cu")
+		(net "+3V3")
+	)
+	(via
+		(at 68.075 6.25)
+		(size 0.5)
+		(drill 0.3)
+		(layers "F.Cu" "B.Cu")
+		(net "+3V3")
+	)
+	(segment
+		(start 31.0294 9.05)
+		(end 30.6294 9.05)
+		(width 0.3)
+		(layer "B.Cu")
+		(net "+3V3")
+	)
+	(segment
+		(start 30.6294 9.05)
+		(end 30.5294 9.05)
+		(width 0.2)
+		(layer "B.Cu")
+		(net "+3V3")
+	)
+	(segment
+		(start 30.945214 23.935)
+		(end 31.395214 23.485)
+		(width 0.3)
+		(layer "B.Cu")
+		(net "+3V3")
+	)
+	(segment
+		(start 31.2294 9.25)
+		(end 31.0294 9.05)
+		(width 0.3)
+		(layer "B.Cu")
+		(net "+3V3")
+	)
+	(segment
+		(start 32.315807 21.868992)
+		(end 32.365807 21.868992)
+		(width 0.2)
+		(layer "B.Cu")
+		(net "I2C_SDA")
+	)
+	(segment
+		(start 32.315807 21.918992)
+		(end 32.315807 21.868992)
+		(width 0.15)
+		(layer "B.Cu")
+		(net "I2C_SDA")
+	)
+	(segment
+		(start 32.715807 21.518992)
+		(end 32.965807 21.518992)
+		(width 0.2)
+		(layer "B.Cu")
+		(net "I2C_SDA")
+	)
+	(segment
+		(start 32.365807 21.868992)
+		(end 32.715807 21.518992)
+		(width 0.2)
+		(layer "B.Cu")
+		(net "I2C_SDA")
+	)
+	(segment
+		(start 32.165807 21.968992)
+		(end 32.215807 21.968992)
+		(width 0.2)
+		(layer "B.Cu")
+		(net "I2C_SDA")
+	)
+	(segment
+		(start 33.265807 21.218992)
+		(end 33.265807 14.168992)
+		(width 0.2)
+		(layer "B.Cu")
+		(net "I2C_SDA")
+	)
+	(segment
+		(start 32.265807 21.918992)
+		(end 32.315807 21.918992)
+		(width 0.15)
+		(layer "B.Cu")
+		(net "I2C_SDA")
+	)
+	(segment
+		(start 33.265807 14.168992)
+		(end 30.515807 11.418992)
+		(width 0.2)
+		(layer "B.Cu")
+		(net "I2C_SDA")
+	)
+	(segment
+		(start 31.965807 22.018992)
+		(end 32.115807 22.018992)
+		(width 0.2)
+		(layer "B.Cu")
+		(net "I2C_SDA")
+	)
+	(segment
+		(start 32.215807 21.968992)
+		(end 32.265807 21.918992)
+		(width 0.2)
+		(layer "B.Cu")
+		(net "I2C_SDA")
+	)
+	(segment
+		(start 32.115807 22.018992)
+		(end 32.165807 21.968992)
+		(width 0.2)
+		(layer "B.Cu")
+		(net "I2C_SDA")
+	)
+	(segment
+		(start 32.965807 21.518992)
+		(end 33.265807 21.218992)
+		(width 0.2)
+		(layer "B.Cu")
+		(net "I2C_SDA")
+	)
+	(segment
+		(start 30.974999 13.05)
+		(end 30.224999 12.3)
+		(width 0.2)
+		(layer "F.Cu")
+		(net "I2C_SCL")
+	)
+	(segment
+		(start 30.224999 12.3)
+		(end 28.525 12.3)
+		(width 0.2)
+		(layer "F.Cu")
+		(net "I2C_SCL")
+	)
+	(via
+		(at 30.974999 13.05)
+		(size 0.5)
+		(drill 0.3)
+		(layers "F.Cu" "B.Cu")
+		(net "I2C_SCL")
+	)
+	(via
+		(at 28.525 12.3)
+		(size 0.5)
+		(drill 0.3)
+		(layers "F.Cu" "B.Cu")
+		(net "I2C_SCL")
+	)
+	(segment
+		(start 32.075 19.15)
+		(end 32.075 14.15)
+		(width 0.2)
+		(layer "B.Cu")
+		(net "I2C_SCL")
+	)
+	(segment
+		(start 32.075 14.15)
+		(end 30.974999 13.05)
+		(width 0.2)
+		(layer "B.Cu")
+		(net "I2C_SCL")
+	)
+	(segment
+		(start 31.875 19.35)
+		(end 32.075 19.15)
+		(width 0.2)
+		(layer "B.Cu")
+		(net "I2C_SCL")
+	)
+	(segment
+		(start 28.525 12.3)
+		(end 28.525 12.1)
+		(width 0.2)
+		(layer "B.Cu")
+		(net "I2C_SCL")
 	)
 	(zone

Commit message: eTutti Viaggio J1 rota restante: lote 4 — bolsoes de +3V3 no teclado
14 +3V3 links, mostly a via (0.5/0.3) from J's B.Cu +3V3 tracks into the
In2 +3V3 pockets, plus short 0.3 tracks. +3V3 now has no open link.
DRC: no new clearance/short/hole; unrouted 28 -> 13.

Co-Authored-By: Claude Opus 5.5 <noreply@anthropic.com>
Routing:
- net +3V3: track 247.5 -> 257.9 mm, vias 51 -> 62
Changed lines of the file:
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@@
 		(net "I2C_SCL")
+	)
+	(segment
+		(start 177.3736 8.05023)
+		(end 178.1236 8.80023)
+		(width 0.3)
+		(layer "F.Cu")
+		(net "+3V3")
+	)
+	(via
+		(at 113.866392 13.3972)
+		(size 0.5)
+		(drill 0.3)
+		(layers "F.Cu" "B.Cu")
+		(net "+3V3")
+	)
+	(via
+		(at 178.1236 8.80023)
+		(size 0.5)
+		(drill 0.3)
+		(layers "F.Cu" "B.Cu")
+		(net "+3V3")
+	)
+	(via
+		(at 98.682992 39.621814)
+		(size 0.5)
+		(drill 0.3)
+		(layers "F.Cu" "B.Cu")
+		(net "+3V3")
+	)
+	(via
+		(at 114.9 41.615)
+		(size 0.5)
+		(drill 0.3)
+		(layers "F.Cu" "B.Cu")
+		(net "+3V3")
+	)
+	(via
+		(at 154.109692 71.673614)
+		(size 0.5)
+		(drill 0.3)
+		(layers "F.Cu" "B.Cu")
+		(net "+3V3")
+	)
+	(via
+		(at 218.850514 55.635)
+		(size 0.5)
+		(drill 0.3)
+		(layers "F.Cu" "B.Cu")
+		(net "+3V3")
+	)
+	(via
+		(at 145.549999 56.934108)
+		(size 0.5)
+		(drill 0.3)
+		(layers "F.Cu" "B.Cu")
+		(net "+3V3")
+	)
+	(via
+		(at 177.3736 8.05023)
+		(size 0.5)
+		(drill 0.3)
+		(layers "F.Cu" "B.Cu")
+		(net "+3V3")
+	)
+	(via
+		(at 200.449495 23.595)
+		(size 0.5)
+		(drill 0.3)
+		(layers "F.Cu" "B.Cu")
+		(net "+3V3")
+	)
+	(via
+		(at 172.7 71.655)
+		(size 0.5)
+		(drill 0.3)
+		(layers "F.Cu" "B.Cu")
+		(net "+3V3")
+	)
+	(via
+		(at 164 25.916292)
+		(size 0.5)
+		(drill 0.3)
+		(layers "F.Cu" "B.Cu")
+		(net "+3V3")
+	)
+	(segment
+		(start 115.9 40.615)
+		(end 114.9 41.615)
+		(width 0.3)
+		(layer "B.Cu")
+		(net "+3V3")
+	)
+	(segment
+		(start 181.834993 24.820365)
+		(end 181.834993 24.870365)
+		(width 0.2)
+		(layer "B.Cu")
+		(net "+3V3")
+	)
+	(segment
+		(start 117.15 40.615)
+		(end 116.9 40.615)
+		(width 0.3)
+		(layer "B.Cu")
+		(net "+3V3")
+	)
+	(segment
+		(start 163.95 25.566292)
+		(end 163.95 25.866292)
+		(width 0.2)
+		(layer "B.Cu")
+		(net "+3V3")
+	)
+	(segment
+		(start 114.216392 13.3972)
+		(end 113.866392 13.3972)
+		(width 0.3)
+		(layer "B.Cu")
+		(net "+3V3")
+	)
+	(segment
+		(start 163.899999 25.516292)
+		(end 163.95 25.566292)
+		(width 0.2)
+		(layer "B.Cu")
+		(net "+3V3")
+	)
+	(segment
+		(start 163.549999 25.366292)
+		(end 163.75 25.366292)
+		(width 0.2)
+		(layer "B.Cu")
+		(net "+3V3")
+	)
+	(segment
+		(start 126.3488 24.087289)
+		(end 125.8488 23.587289)
+		(width 0.3)
+		(layer "B.Cu")
+		(net "+3V3")
+	)
+	(segment
+		(start 164.302729 24.439689)
+		(end 164.302729 24.839689)
+		(width 0.2)
+		(layer "B.Cu")
+		(net "+3V3")
+	)
+	(segment
+		(start 126.3488 24.887289)
+		(end 126.3488 24.087289)
+		(width 0.2)
+		(layer "B.Cu")
+		(net "+3V3")
+	)
+	(segment
+		(start 163.75 25.366292)
+		(end 163.899999 25.516292)
+		(width 0.3)
+		(layer "B.Cu")
+		(net "+3V3")
+	)
+	(segment
+		(start 116.9 40.615)
+		(end 115.9 40.615)
+		(width 0.2)
+		(layer "B.Cu")
+		(net "+3V3")
+	)
+	(segment
+		(start 163.952729 23.889689)
+		(end 164.302729 24.239689)
+		(width 0.3)
+		(layer "B.Cu")
+		(net "+3V3")
+	)
+	(segment
+		(start 164.302729 24.239689)
+		(end 164.302729 24.439689)
+		(width 0.3)
+		(layer "B.Cu")
+		(net "+3V3")
+	)
+	(segment
+		(start 163.95 25.866292)
+		(end 164 25.916292)
+		(width 0.3)
+		(layer "B.Cu")
+		(net "+3V3")
+	)
+	(segment
+		(start 164.302729 24.839689)
+		(end 164.252729 24.889689)
+		(width 0.3)
+		(layer "B.Cu")
+		(net "+3V3")
+	)
+	(segment
+		(start 145.049999 56.934108)
+		(end 145.549999 56.934108)
+		(width 0.3)
+		(layer "B.Cu")
+		(net "+3V3")
+	)
+	(segment
+		(start 164.252729 24.889689)
+		(end 163.852729 25.289689)
+		(width 0.2)
+		(layer "B.Cu")
+		(net "+3V3")
+	)
+	(segment
+		(start 181.834993 23.270365)
+		(end 181.834993 24.820365)
+		(width 0.3)
+		(layer "B.Cu")
+		(net "+3V3")
+	)
+	(segment
+		(start 144.5567 59.985)
+		(end 144.5567 59.935)
+		(width 0.3)
+		(layer "In2.Cu")
+		(net "+3V3")
 	)
 	(zone
