File: etutti/hardware/viaggio_j1/kicad/viaggio_micromod.kicad_pcb (KiCad board)
At the start: 4 copper layers, 246.5 x 95 mm, 177 parts, among them J101 91302-42-067RCE, J201 TYPE-C-31-M-12, J202 S3B-PH-SM4-TB, J301 PJ-327A 5JJ, J501 alto-falante (fios), Q201 AO3401A, Q202 AO3400A, Q203 AO3401A, SW1 Gateron_Magnetic_MX_1u, SW10 Gateron_Magnetic_MX_1u, SW11 Gateron_Magnetic_MX_1u, SW12 Gateron_Magnetic_MX_1u, SW13 Gateron_Magnetic_MX_1u, SW14 Gateron_Magnetic_MX_1u, SW15 Gateron_Magnetic_MX_1u, SW16 Gateron_Magnetic_MX_1u, SW17 Gateron_Magnetic_MX_1u, SW18 Gateron_Magnetic_MX_1u, SW19 Gateron_Magnetic_MX_1u, SW2 Gateron_Magnetic_MX_1u, SW20 Gateron_Magnetic_MX_1u, SW21 Gateron_Magnetic_MX_1u, SW22 Gateron_Magnetic_MX_1u, SW23 Gateron_Magnetic_MX_1u, SW24 Gateron_Magnetic_MX_1u, SW25 Gateron_Magnetic_MX_1u, SW26 Gateron_Magnetic_MX_1u, SW27 Gateron_Magnetic_MX_1u, SW28 Gateron_Magnetic_MX_1u, SW3 Gateron_Magnetic_MX_1u, SW4 Gateron_Magnetic_MX_1u, SW401 EC11E18244A5, SW402 EC11E18244A5, SW403 Program, SW5 Gateron_Magnetic_MX_1u, SW6 Gateron_Magnetic_MX_1u, SW7 Gateron_Magnetic_MX_1u, SW8 Gateron_Magnetic_MX_1u, SW9 Gateron_Magnetic_MX_1u, U201 USBLC6-2SC6, U202 BQ24074RGTR, U203 74LVC1G08, U204 TPS63001DRCR, U301 SGTL5000XNLA3, U302 XC6206P182MR, U501 MAX98357AETE+T, U601 74HC4067PW, U602 74HC4067PW, U603 74LVC1G04, U604 74LVC1G08, U605 74LVC1G08, U701 TMAG5253BA3IQDMRR, U702 TMAG5253BA3IQDMRR, U703 TMAG5253BA3IQDMRR, U704 TMAG5253BA3IQDMRR, U705 TMAG5253BA3IQDMRR, U706 TMAG5253BA3IQDMRR, U707 TMAG5253BA3IQDMRR, U708 TMAG5253BA3IQDMRR, U709 TMAG5253BA3IQDMRR, U710 TMAG5253BA3IQDMRR, U711 TMAG5253BA3IQDMRR, U712 TMAG5253BA3IQDMRR, U713 TMAG5253BA3IQDMRR, U714 TMAG5253BA3IQDMRR, U715 TMAG5253BA3IQDMRR, U716 TMAG5253BA3IQDMRR, U717 TMAG5253BA3IQDMRR, U718 TMAG5253BA3IQDMRR, U719 TMAG5253BA3IQDMRR, U720 TMAG5253BA3IQDMRR, U721 TMAG5253BA3IQDMRR, U722 TMAG5253BA3IQDMRR, U723 TMAG5253BA3IQDMRR, U724 TMAG5253BA3IQDMRR, U725 TMAG5253BA3IQDMRR, U726 TMAG5253BA3IQDMRR, U727 TMAG5253BA3IQDMRR, U728 TMAG5253BA3IQDMRR

Commit message: eTutti Viaggio J1 fechamento: lote 6b — codec
Two GND vias 0.5/0.3 in the codec's exposed pad U301.21, at (24.00; 35.50)
and (23.45; 34.95). The In2 track of I2S_BCLK under the pad (13.7 mm) was
taken out and remade between the same two points: 21.1 mm, 0.2, In2/F/B,
2 vias. Detour end points on a via may now leave on any layer.

Counts from the KiCad DRC (--schematic-parity --severity-all):
- before: track_width 13, unconnected 6 (GND 3, VSYS 2, BB_L1 1), parity 0
- after: track_width 13 (J's), unconnected 5 (GND 2, VSYS 2, BB_L1 1),
  parity 0; no clearance/short/hole/dangling violations
- GND left: C304.2 (no way out even without the In2 tracks) and R209.2
  (its 6a link was cut loose by the zone refill; retried in 6c)

Co-Authored-By: Claude Opus 5.5 <noreply@anthropic.com>
Routing:
- net I2S_BCLK: track 85.2 -> 92.6 mm, vias 3 -> 5
- net GND: vias 947 -> 949
Changed lines of the file:
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@@
 	)
 	(segment
-		(start 22.5109 34.2446)
-		(end 32.1752 43.9089)
-		(width 0.2)
-		(layer "In2.Cu")
-		(net "I2S_BCLK")
-	)
-	(segment
 		(start 32.1752 43.9089)
 		(end 32.1752 61.782)
@@
 		(net "USB_HOLD")
 	)
+	(via
+		(at 23.45 34.95)
+		(size 0.5)
+		(drill 0.3)
+		(layers "F.Cu" "B.Cu")
+		(net "GND")
+	)
+	(via
+		(at 24 35.5)
+		(size 0.5)
+		(drill 0.3)
+		(layers "F.Cu" "B.Cu")
+		(net "GND")
+	)
+	(segment
+		(start 22.4609 34.1446)
+		(end 22.1109 33.794599)
+		(width 0.2)
+		(layer "F.Cu")
+		(net "I2S_BCLK")
+	)
+	(segment
+		(start 21.3109 33.794599)
+		(end 20.910899 34.1946)
+		(width 0.2)
+		(layer "F.Cu")
+		(net "I2S_BCLK")
+	)
+	(segment
+		(start 22.1109 33.794599)
+		(end 21.3109 33.794599)
+		(width 0.2)
+		(layer "F.Cu")
+		(net "I2S_BCLK")
+	)
+	(segment
+		(start 22.5109 34.2446)
+		(end 22.4609 34.1446)
+		(width 0.2)
+		(layer "F.Cu")
+		(net "I2S_BCLK")
+	)
+	(segment
+		(start 20.910899 34.1946)
+		(end 19.9609 34.1946)
+		(width 0.2)
+		(layer "F.Cu")
+		(net "I2S_BCLK")
+	)
+	(via
+		(at 32.1109 43.7946)
+		(size 0.5)
+		(drill 0.3)
+		(layers "F.Cu" "B.Cu")
+		(net "I2S_BCLK")
+	)
+	(via
+		(at 19.9609 34.1946)
+		(size 0.5)
+		(drill 0.3)
+		(layers "F.Cu" "B.Cu")
+		(net "I2S_BCLK")
+	)
+	(segment
+		(start 19.410899 34.7446)
+		(end 19.410899 36.1946)
+		(width 0.2)
+		(layer "B.Cu")
+		(net "I2S_BCLK")
+	)
+	(segment
+		(start 27.0109 43.7946)
+		(end 32.1109 43.7946)
+		(width 0.2)
+		(layer "B.Cu")
+		(net "I2S_BCLK")
+	)
+	(segment
+		(start 19.410899 36.1946)
+		(end 27.0109 43.7946)
+		(width 0.2)
+		(layer "B.Cu")
+		(net "I2S_BCLK")
+	)
+	(segment
+		(start 19.9609 34.1946)
+		(end 19.410899 34.7446)
+		(width 0.2)
+		(layer "B.Cu")
+		(net "I2S_BCLK")
+	)
+	(segment
+		(start 32.1109 43.7946)
+		(end 32.175199 43.9089)
+		(width 0.2)
+		(layer "In2.Cu")
+		(net "I2S_BCLK")
+	)
 	(zone

Commit message: eTutti Viaggio J1 fechamento: lote 6c — o que restou
R209.2 (GND), cut loose again by the 6a zone refill, now goes down to the
In1 plane by its own via at (67.63; 18.53). In 6c the power tracks within
5 mm of U202.10/11 could also be ripped; still no way out.

Counts from the KiCad DRC (--schematic-parity --severity-all):
- before: track_width 13, unconnected 5 (GND 2, VSYS 2, BB_L1 1), parity 0
- after: track_width 13 (J's), unconnected 4 (GND 1, VSYS 2, BB_L1 1),
  parity 0; no clearance/short/hole/dangling violations
- left out after 2 attempts each: GND C304.2, VSYS U202.10/11,
  VSYS U204.5, BB_L1 U204.4-L201.1 (reasons in COBRE.md)

Co-Authored-By: Claude Opus 5.5 <noreply@anthropic.com>
Routing:
- net GND: vias 949 -> 950
Changed lines of the file:
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@@
 		(net "I2S_BCLK")
+	)
+	(via
+		(at 67.313192 19.6755)
+		(size 0.5)
+		(drill 0.3)
+		(layers "F.Cu" "B.Cu")
+		(net "GND")
 	)
 	(zone
