File: etutti/hardware/viaggio_j1/kicad/viaggio_micromod_E.kicad_sch (KiCad schematic)
At the start: 43 parts, among them J201 TYPE-C-31-M-12, J202 S3B-PH-SM4-TB, Q201 AO3401A, Q202 AO3400A, Q203 AO3401A, U201 USBLC6-2SC6, U202 BQ24074RGTR, U203 74LVC1G08, U204 TPS63001DRCR

Commit message: eTutti Viaggio J1 M3: lote 1 — C202/C206, C210 de VSYS, C207, via do C304
- C202 (E3) and C206 (E4) swap places on the board, so each reference sits where its
  schematic function is (same 10 uF 0805, same nets); the schematic is unchanged for them.
- C210 (new, 10 uF 0603 C19702, E3): VSYS cap at U202's OUT pins, on the top side (no room
  on the back); added to viaggio_micromod/pcb/schematic.py, sheet E copied to the J1 project.
- C207 next to C208 (3.55 mm), its old vias out.
- C304: GND via out of the pad; J's +3V3 loop C305.1-C304.1 redone at 0.2 and C304 moved
  0.59 mm into the room it left.
- m3.py (lote1): splice save as energia.py, 4008 blocks checked identical.

DRC: track_width 7 (J's, unchanged), 0 clearance/short/hole, 0 unconnected, parity 0. ERC 0/0.

Co-Authored-By: Claude Opus 5.5 <noreply@anthropic.com>
Parts:
- added C210: 10uF, Capacitor_SMD:C_0603_1608Metric, symbol viaggio_micromod:C
Connections:
- net GND: now also C210.2
- net VSYS: now also C210.1
Other:
- moved on the sheet: C204, C205, C206, C207, C208, C209, C213, D202, D203, D204, D205, J202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
