File: etutti/hardware/viaggio_j1/kicad/viaggio_micromod_A.kicad_sch (KiCad schematic)
At the start: 5 parts, among them J501 alto-falante (fios), U501 MAX98357AETE+T

Commit message: eTutti Viaggio J1 M3b: LCSC codes, board-name silkscreen, SW403 height, fab/ with ENIG
- C307 (150 nF 0402 X7R 16 V, VAG): Murata GRM155R71C154KA12D, LCSC C162182;
  FB301 C1002 and R501 C4131 now in schematic.py (sheets F and A), the J1
  sheets and the board's LCSC fields
- silkscreen top and bottom: "eTutti Viaggio MicroMod · J1 · SPEC v2.5"
- SW403 Altura_mm 20 -> 1.5; build_board.py HEIGHT_MM matches SW403 before SW40
- m3.py m3b: only 6 blocks rewritten (one line each); tracks, vias, zones and
  footprint positions checked identical by uuid; lote3 --sem-plate; BOM fails
  on a part without LCSC code; ENIG recorded in the order parameters
- fab/: Gerbers (only silkscreen changed), BOM, renders; CPL and plate unchanged
- DRC: 0 clearance/short/hole/silk, 0 unconnected, parity 0, only the 3
  accepted EN_B track_width; ERC 0

Co-Authored-By: Claude Opus 5.5 <noreply@anthropic.com>
Parts:
- R501: LCSC (none) -> C4131
Changed lines of the file:
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@@
 		(property "Description" "com os 100k internos: 0,42 V no SD_MODE = (L+R)/2; pino baixo = desligado" (at 88.9 48.26 0) (hide yes) (effects (font (size 1.27 1.27))))
 		(property "Codigo" "A1" (at 92.71 44.45 0) (effects (font (size 1.27 1.27)) (justify right)))
-		(property "LCSC" "" (at 88.9 48.26 0) (hide yes) (effects (font (size 1.27 1.27))))
+		(property "LCSC" "C4131" (at 88.9 48.26 0) (hide yes) (effects (font (size 1.27 1.27))))
 		(property "Montagem" "JLC" (at 88.9 48.26 0) (hide yes) (effects (font (size 1.27 1.27))))
 		(pin "1")
